Commit message: teo_control temporal file added

File: teo_description/urdf/others/teo_transmission.xacro (robot description, xacro)
@@ -8,7 +8,8 @@
 		<transmission name="${side}_${name}_${axis}_trans">
 			<type>transmission_interface/SimpleTransmission</type>
-			<joint name="${side}_${name}_${axis}"/>
+			<joint name="${side}_${name}_${axis}">
+				<hardwareInterface>EffortJointInterface</hardwareInterface>
+      </joint>
 			<actuator name="${side}_${name}_${axis}_motor" >
-				<hardwareInterface>EffortJointInterface</hardwareInterface>
 				<mechanicalReduction>${reduction}</mechanicalReduction>
 			</actuator>
@@ -18,7 +19,8 @@
 		<transmission name="waist_${axis}_trans">
 			<type>transmission_interface/SimpleTransmission</type>
-			<joint name="waist_${axis}" />
+			<joint name="waist_${axis}">
+				<hardwareInterface>EffortJointInterface</hardwareInterface>
+      </joint>
 			<actuator name="waist_${axis}_motor" >
-				<hardwareInterface>EffortJointInterface</hardwareInterface>
 				<mechanicalReduction>${reduction}</mechanicalReduction>
 			</actuator>
