Commit message: custom materials for teo_gazebo

File: teo_description/urdf/teo_structure.gazebo.xacro (robot description, xacro)
@@ -14,10 +14,10 @@
 			<mu1>0.9</mu1>
 			<mu2>0.9</mu2>
-			<material>Gazebo/White</material>
+			<!-- <material>Gazebo/White</material> -->
 		</gazebo>
 		<gazebo reference="waist_pitch_link">
 			<mu1>0.9</mu1>
 			<mu2>0.9</mu2>
-			<material>Gazebo/White</material>
+			<!-- <material>Gazebo/White</material> -->
 		</gazebo>
 <!-- 		<gazebo reference="waist">
@@ -34,25 +34,25 @@
 			<mu1>0.9</mu1>
 			<mu2>0.9</mu2>
-			<material>Gazebo/White</material>
+			<!-- <material>Gazebo/White</material> -->
 		</gazebo>
 		<gazebo reference="${side}_hip_yaw_link">
 			<mu1>0.9</mu1>
 			<mu2>0.9</mu2>
-			<material>Gazebo/White</material>
+			<!-- <material>Gazebo/White</material> -->
 		</gazebo>
 		<gazebo reference="${side}_femur_link">
 			<mu1>0.9</mu1>
 			<mu2>0.9</mu2>
-			<material>Gazebo/White</material>
+			<!-- <material>Gazebo/White</material> -->
 		</gazebo>
 		<gazebo reference="${side}_tibia_link">
 			<mu1>0.9</mu1>
 			<mu2>0.9</mu2>
-			<material>Gazebo/White</material>
+			<!-- <material>Gazebo/White</material> -->
 		</gazebo>
 		<gazebo reference="${side}_ankle_pitch_link">
 			<mu1>0.9</mu1>
 			<mu2>0.9</mu2>
-			<material>Gazebo/White</material>
+			<!-- <material>Gazebo/White</material> -->
 		</gazebo>
 		<gazebo reference="${side}_astragalus_link">
@@ -65,5 +65,5 @@
 			<minDepth>0.00</minDepth>
 			<implicitSpringDamper>1</implicitSpringDamper>
-			<material>Gazebo/White</material>
+			<!-- <material>Gazebo/White</material> -->
 		</gazebo>
 		<gazebo reference="${side}_sole">
@@ -73,5 +73,5 @@
 	    <maxVel>1.0</maxVel>
 	    <minDepth>0.003</minDepth>
-	    <material>Gazebo/White</material>
+	    <!-- <material>Gazebo/White</material> -->
 		</gazebo>
   </xacro:macro>
