Commit message: new visualization for teo_description

File: teo_description/urdf/arms/arm.urdf.xacro (robot description, xacro)
@@ -10,9 +10,9 @@
 <!-- *** TEO ARM PARAMETERS -->
 <!-- Link lengths (meters)-->
-	<xacro:property name="chest_link1" value="0.0" />
-	<xacro:property name="chest_link2" value="0.245" />
+	<!--xacro:property name="chest_link1" value="0.0" />
+	<xacro:property name="chest_link2" value="0.245" /-->
 	<xacro:property name="arm_link1" value="0.340" /> <!-- Clavicle -->
-	<xacro:property name="arm_link2" value="0.337" /> <!-- Humerus -->
-	<xacro:property name="arm_link3" value="0.210" /> <!-- Ulna -->
+	<xacro:property name="arm_link2" value="0.32901" /> <!-- Humerus -->
+	<xacro:property name="arm_link3" value="0.202" /> <!-- Ulna -->
 <!-- Minimum angles (degrees) -->
 	<xacro:property name="shoulder_pitch_lower" value="${-180 * deg_to_rad}" />
@@ -76,4 +76,5 @@
 					izz="1.000" />
       </inertial>
+      <xacro:insert_visualization_shoulder_pitch side="${side}" reflect="${reflect}"/>
     </link>
     <link name="${side}_shoulder_roll_link">
@@ -86,4 +87,5 @@
 					izz="1.000" />
       </inertial>
+      <xacro:insert_visualization_shoulder_roll side="${side}" reflect="${reflect}"/>
     </link>
     <link name="${side}_shoulder_yaw_link">
@@ -118,4 +120,5 @@
 					izz="1.000" />
       </inertial>
+      <xacro:insert_visualization_wrist_yaw side="${side}" reflect="${reflect}"/>
     </link>
     <link name="${side}_wrist_pitch_link">
@@ -128,4 +131,5 @@
 					izz="1.525e-4" />
       </inertial>
+      <xacro:insert_visualization_wrist_pitch side="${side}" reflect="${reflect}"/>
     </link>
   </xacro:macro>
@@ -135,5 +139,5 @@
       <parent link="waist_pitch_link"/>
       <child link="${side}_shoulder_pitch_link"/>
-      <origin xyz="-${chest_link1} ${reflect*arm_link1} ${chest_link2}" rpy="0 0 0"/>
+      <origin xyz="-${chest_link1} ${reflect*arm_link1} ${chest_link2+torso_link2}" rpy="0 0 0"/>
       <axis xyz="0 1 0"/>
       <limit velocity="${shoulder_pitch_velocity}" effort="${shoulder_pitch_effort}" lower="${shoulder_pitch_lower}" upper="${shoulder_pitch_upper}"/>

File: teo_description/urdf/arms/arms_vis.urdf.xacro (robot description, xacro)
@@ -7,10 +7,10 @@
 <robot xmlns:xacro="http://ros.org/wiki/xacro">
   <xacro:macro name="insert_visualization_shoulder_pitch" params="side reflect">
-    <!--visual>
+    <visual>
+      <origin rpy="0 0 0" xyz="0 0 0"/>
       <geometry>
-        <box size="0.1 ${arm_link1} 0.1"/>
+        <mesh filename="package://teo_description/meshes/arms/${side}_shoulder_pitch.stl"/>
       </geometry>
-      <material name="grey"/>
-      <origin rpy="0 0 0" xyz="${chest_link1} ${arm_link1/2*reflect} ${chest_link2}"/>
+      <material name="teoGray"/>
     </visual>
     <collision>
@@ -18,17 +18,43 @@
         <box size="0.1 ${arm_link1} 0.1"/>
       </geometry>
-      <origin rpy="0 0 0" xyz="${chest_link1} ${arm_link1/2*reflect} ${chest_link2}"/>
-    </collision-->
+      <origin rpy="0 0 0" xyz="0 0 0"/>
+    </collision>
+  </xacro:macro>
+  <xacro:macro name="insert_visualization_shoulder_roll" params="side reflect">
+    <visual>
+      <origin rpy="0 0 0" xyz="0 0 0"/>
+      <geometry>
+        <mesh filename="package://teo_description/meshes/arms/${side}_shoulder_roll.stl"/>
+      </geometry>
+      <material name="teoGray"/>
+    </visual>
+    <collision>
+      <geometry>
+        <box size="0.1 ${arm_link1} 0.1"/>
+      </geometry>
+      <origin rpy="0 0 0" xyz="0 0 0"/>
+    </collision>
   </xacro:macro>
   <xacro:macro name="insert_visualization_shoulder_yaw" params="side reflect">
     <visual>
+      <origin rpy="0 0 0" xyz="0 0 -0.12126"/>
       <geometry>
-        <!--box size="0.08 0.08 ${arm_link2}"/-->
-        <!--mesh filename="package://teo_description/meshes/legs/${side}_foot.dae"/-->
-        <mesh filename="package://teo_description/meshes/arms/${side}_arm.dae"/>
+        <mesh filename="package://teo_description/meshes/arms/${side}_shoulder_yaw.stl"/>
       </geometry>
-      <material name="grey"/>
-      <!--origin rpy="0 0 0" xyz="0 0 -${arm_link2/2}"/-->
-      <origin rpy="0 0 0" xyz="0 0 -${arm_link2/2-0.045}"/>
+      <material name="teoGray"/>
+    </visual>
+    <visual>
+      <origin rpy="0 0 0" xyz="0 0 -0.27651"/>
+      <geometry>
+        <mesh filename="package://teo_description/meshes/arms/${side}_humerus.stl"/>
+      </geometry>
+      <material name="teoGray"/>
+    </visual>
+    <visual>
+      <origin rpy="0 0 0" xyz="0 0 -0.28351"/>
+      <geometry>
+        <mesh filename="package://teo_description/meshes/arms/${side}_union_humerus_elbow.stl"/>
+      </geometry>
+      <material name="teoGray"/>
     </visual>
     <collision>
@@ -41,10 +67,22 @@
   <xacro:macro name="insert_visualization_elbow_pitch" params="side reflect">
     <visual>
+      <origin rpy="0 0 0" xyz="0 0 0"/>
       <geometry>
-        <!--box size="0.06 0.06 ${arm_link3}"/-->
-        <mesh filename="package://teo_description/meshes/arms/${side}_forearm.dae"/>
+        <mesh filename="package://teo_description/meshes/arms/${side}_elbow_pitch.stl"/>
       </geometry>
-      <material name="grey"/>
-      <origin rpy="0 0 0" xyz="0 0 -${arm_link3/2}"/>
+      <material name="teoGray"/>
+    </visual>
+    <visual>
+      <origin rpy="0 0 0" xyz="0 0 -0.11324"/>
+      <geometry>
+        <mesh filename="package://teo_description/meshes/arms/${side}_elbow_link.stl"/>
+      </geometry>
+    </visual>
+    <visual>
+      <origin rpy="0 0 0" xyz="0 0 -0.11324"/>
+      <geometry>
+        <mesh filename="package://teo_description/meshes/arms/${side}_union_elbow_wrist.stl"/>
+      </geometry>
+      <material name="teoGray"/>
     </visual>
     <collision>
@@ -55,3 +93,47 @@
     </collision>
   </xacro:macro>
+  <xacro:macro name="insert_visualization_wrist_yaw" params="side reflect">
+    <visual>
+      <origin rpy="0 0 0" xyz="0 0 0"/>
+      <geometry>
+        <mesh filename="package://teo_description/meshes/arms/${side}_wrist_yaw.stl"/>
+      </geometry>
+      <material name="teoGray"/>
+    </visual>
+    <collision>
+      <geometry>
+        <box size="0.03 0.03 0.03"/>
+      </geometry>
+      <origin rpy="0 0 0" xyz="0 0 -0.015"/>
+    </collision>
+  </xacro:macro>
+  <xacro:macro name="insert_visualization_wrist_pitch" params="side reflect">
+    <visual>
+      <origin rpy="0 0 0" xyz="0 0 0"/>
+      <geometry>
+        <mesh filename="package://teo_description/meshes/arms/${side}_wrist_pitch.stl"/>
+      </geometry>
+      <material name="teoGray"/>
+    </visual>
+    <visual>
+      <origin rpy="0 0 0" xyz="0 0 -0.056"/>
+      <geometry>
+        <mesh filename="package://teo_description/meshes/arms/${side}_wrist_sensorFT.stl"/>
+      </geometry>
+      <material name="teoGray"/>
+    </visual>
+    <visual>
+      <origin rpy="0 0 0" xyz="0 0 -0.056"/>
+      <geometry>
+        <mesh filename="package://teo_description/meshes/arms/${side}_hand.stl"/>
+      </geometry>
+      <material name="teoGray"/>
+    </visual>
+    <collision>
+      <geometry>
+        <box size="0.03 0.03 0.03"/>
+      </geometry>
+      <origin rpy="0 0 0" xyz="0 0 -0.015"/>
+    </collision>
+  </xacro:macro>
 </robot>

File: teo_description/urdf/legs/leg.urdf.xacro (robot description, xacro)
@@ -10,4 +10,5 @@
 <!-- *** TEO LEG PARAMETERS -->
 <!-- Link lengths -->
+	<xacro:property name="leg_link0" value="0.10237" /> <!-- Hip -->
 	<xacro:property name="leg_link1" value="0.146" /> <!-- Hip -->
 	<xacro:property name="leg_link2" value="0.33" /> <!-- Femur -->
@@ -76,4 +77,5 @@
 					izz="0.001" />
       </inertial>
+			<xacro:insert_visualization_hip_yaw side="${side}" reflect="{reflect}"/>
     </link>
     <link name="${side}_hip_roll_link">
@@ -86,5 +88,5 @@
 					izz="0.000001" />
       </inertial>
-			<xacro:insert_visualization_hip_roll side="${side}" reflect="{reflect}"/>
+			<xacro:insert_visualization_hip_pitch side="${side}" reflect="{reflect}"/>
     </link>
     <link name="${side}_femur_link">
@@ -130,6 +132,5 @@
           izz="0.000006" />
       </inertial>
-      <xacro:insert_visualization_astragalus_link side="${side}" reflect="${reflect}"/>
-      <xacro:insert_visualization_sole side="${side}" reflect="${reflect}"/> <!-- OJO, falta bajarlo -link5/2-->
+      <xacro:insert_visualization_ankle_roll side="${side}" reflect="${reflect}"/>
     </link>
     <link name="${side}_sole">
@@ -142,4 +143,6 @@
 					izz="0.001" />
       </inertial>
+      <xacro:insert_visualization_foot side="${side}" reflect="${reflect}"/>
+      <xacro:insert_visualization_union_sensorFT_foot side="${side}" reflect="${reflect}"/>
     </link>
   </xacro:macro>
@@ -149,5 +152,5 @@
       <parent link="waist"/>
       <child link="${side}_hip_yaw_link"/>
-      <origin xyz="0 ${reflect*leg_link1} 0" rpy="0 0 0"/> <!--y=Leg_link1-->
+      <origin xyz="0 ${reflect*leg_link1} ${-leg_link0}" rpy="0 0 0"/> <!--y=Leg_link1-->
       <axis xyz="0 0 1"/>
       <limit velocity="${hip_yaw_velocity}" effort="${hip_yaw_effort}" lower="${hip_yaw_lower}" upper="${hip_yaw_upper}"/>

File: teo_description/urdf/legs/legs_vis.urdf.xacro (robot description, xacro)
@@ -8,12 +8,12 @@
   <xacro:macro name="insert_visualization_hip_yaw" params="side reflect">
     <visual>
+      <origin rpy="0 0 0" xyz="0 0 0"/>
       <geometry>
-        <mesh filename="package://teo_description/meshes/legs/${side}_axialhip.dae"/>
+        <mesh filename="package://teo_description/meshes/legs/${side}_hip_yaw.stl"/>
       </geometry>
-      <material name="grey"/>
-      <origin rpy="0 0 0" xyz="0 ${reflect*leg_link1} 0"/>
+      <material name="teoGray"/>
     </visual>
     <collision>
-      <origin xyz="0 ${reflect*leg_link1} 0.045" rpy="0 1.571 0"/>
+      <origin xyz="0 0 0.045" rpy="0 1.571 0"/>
       <geometry>
         <cylinder radius="0.045" length="0.13"/>
@@ -21,20 +21,20 @@
     </collision>
   </xacro:macro>
-  <xacro:macro name="insert_visualization_hip_roll" params="side reflect">
+  <xacro:macro name="insert_visualization_hip_pitch" params="side reflect">
     <visual>
+      <origin rpy="0 0 0" xyz="0 0 0"/>
       <geometry>
-        <mesh filename="package://teo_description/meshes/legs/${side}_hip.dae"/>
+        <mesh filename="package://teo_description/meshes/legs/${side}_hip_pitch.stl"/>
       </geometry>
-      <material name="grey"/>
-      <origin rpy="0 0 0" xyz="0 0 0"/>
+      <material name="teoGray"/>
     </visual>
   </xacro:macro>
   <xacro:macro name="insert_visualization_femur_link" params="side reflect">
     <visual>
+      <origin rpy="0 0 0" xyz="0 0 0"/>
       <geometry>
-        <mesh filename="package://teo_description/meshes/legs/${side}_thigh.dae"/>
+        <mesh filename="package://teo_description/meshes/legs/${side}_femur.stl"/>
       </geometry>
-      <material name="grey"/>
-      <origin rpy="0 0 0" xyz="0.013 0 -${leg_link2}"/>
+      <material name="teoGray"/>
     </visual>
     <collision>
@@ -47,9 +47,9 @@
   <xacro:macro name="insert_visualization_tibia_link" params="side reflect">
     <visual>
+      <origin rpy="0 0 0" xyz="0.0 0.0 0.0"/>
       <geometry>
-        <mesh filename="package://teo_description/meshes/legs/${side}_tibia.dae"/>
+        <mesh filename="package://teo_description/meshes/legs/${side}_tibia.stl"/>
       </geometry>
-      <material name="grey"/>
-      <origin rpy="0 0 0" xyz="-0.013 ${reflect*-(leg_link4)} -${leg_link3}"/>
+      <material name="teoGray"/>
     </visual>
     <collision>
@@ -62,18 +62,33 @@
   <xacro:macro name="insert_visualization_ankle_pitch" params="side reflect">
     <visual>
+      <origin rpy="0 0 0" xyz="0 0 0"/>
       <geometry>
-        <mesh filename="package://teo_description/meshes/legs/${side}_ankle.dae"/>
+        <mesh filename="package://teo_description/meshes/legs/${side}_ankle_pitch.stl"/>
       </geometry>
-      <material name="grey"/>
-      <origin rpy="0 0 0" xyz="0 0 0"/>
+      <material name="teoGray"/>
     </visual>
   </xacro:macro>
-  <xacro:macro name="insert_visualization_astragalus_link" params="side reflect">
+  <xacro:macro name="insert_visualization_ankle_roll" params="side reflect">
     <visual>
+      <origin rpy="0 0 0" xyz="0 0 0"/>
       <geometry>
-        <mesh filename="package://teo_description/meshes/legs/${side}_foot.dae"/>
+        <mesh filename="package://teo_description/meshes/legs/${side}_ankle_roll.stl"/>
       </geometry>
-      <material name="grey"/>
+      <material name="teoGray"/>
+    </visual>
+    <visual>
+      <origin rpy="0 0 0" xyz="0 0 -0.073"/>
+      <geometry>
+        <mesh filename="package://teo_description/meshes/legs/${side}_ankle_sensorFT.stl"/>
+      </geometry>
+    </visual>
+  </xacro:macro>
+  <xacro:macro name="insert_visualization_foot" params="side reflect">
+    <visual>
       <origin rpy="0 0 0" xyz="0 0 0"/>
+      <geometry>
+        <mesh filename="package://teo_description/meshes/legs/${side}_foot.stl"/>
+      </geometry>
+      <material name="teoGray"/>
     </visual>
     <collision>
@@ -83,4 +98,13 @@
       <origin rpy="0 0 0" xyz="0 0 -${leg_link5/2}"/>
     </collision>
+  </xacro:macro>
+  <xacro:macro name="insert_visualization_union_sensorFT_foot" params="side reflect">
+    <visual>
+      <origin rpy="0 0 0" xyz="0 0 0"/>
+      <geometry>
+        <mesh filename="package://teo_description/meshes/legs/${side}_union_sensorFT_foot.stl"/>
+      </geometry>
+      <material name="teoBlue"/>
+    </visual>
   </xacro:macro>
   <xacro:macro name="insert_visualization_sole" params="side reflect">

File: teo_description/urdf/others/teo_colors.xacro (robot description, xacro)
@@ -1,10 +1,16 @@
 <?xml version="1.0"?>
 <!--
-  ROS xacro constants used in the generation of TEO humanoid robot URDF using xacro
+  ROS xacro colors used in the generation of TEO humanoid robot URDF using xacro
   RoboticsLab, University Carlos III of Madrid
 -->
 <robot xmlns:xacro="http://ros.org/wiki/xacro">
- <property name="deg_to_rad" value="0.01745329251994329577" />
- <property name="pi" value="3.1415926535897931"/>
- <property name="pi_2" value="1.5707963267948966"/>
+  <material name="teoGray">
+    <color rgba="0.6 0.6 0.6 1.0"/>
+  </material>
+  <material name="teoBlue">
+    <color rgba="0.0 0.0 1.0 1.0"/>
+  </material>
+  <material name="teoBlack">
+    <color rgba="0.0 0.0 0.0 1.0"/>
+  </material>
 </robot>

File: teo_description/urdf/teo_humanoid.urdf.xacro (robot description, xacro)
@@ -21,4 +21,5 @@
   </xacro:unless-->
   <!--xacro:include filename="$(find teo_description)/urdf/visual.xacro" /-->
+  <xacro:include filename="$(find teo_description)/urdf/others/teo_colors.xacro" />
   <xacro:include filename="$(find teo_description)/urdf/torso/torso_vis.urdf.xacro" />
   <xacro:include filename="$(find teo_description)/urdf/legs/legs_vis.urdf.xacro" />

File: teo_description/urdf/torso/torso.urdf.xacro (robot description, xacro)
@@ -11,7 +11,11 @@
 <!-- Link lengths -->
 	<xacro:property name="waist_link1" value="0.0" />
-	<xacro:property name="waist_link2" value="0.287" />
+	<!--xacro:property name="waist_link2" value="0.287" /-->
+	<xacro:property name="waist_link2" value="0.19070" />
 	<xacro:property name="torso_link1" value="0.0" />
+	<!--xacro:property name="torso_link2" value="0.06" /-->
 	<xacro:property name="torso_link2" value="0.06" />
+  <xacro:property name="chest_link1" value="0.0" />
+  <xacro:property name="chest_link2" value="0.245" />
 <!-- Minimum angles -->
 	<xacro:property name="waist_yaw_lower" value="${-45 * deg_to_rad}" />
@@ -47,6 +51,4 @@
     </inertial>
     <xacro:insert_visualization_waist/>
-    <xacro:insert_visualization_hip_yaw side="r" reflect="-1"/>
-    <xacro:insert_visualization_hip_yaw side="l" reflect="1"/>
   </link>
   <link name="waist_yaw_link" >

File: teo_description/urdf/torso/torso_vis.urdf.xacro (robot description, xacro)
@@ -6,15 +6,11 @@
 -->
 <robot xmlns:xacro="http://ros.org/wiki/xacro">
-  <material name="LightGrey">
-    <color rgba="0.8 0.8 0.8 1.0"/>
-  </material>
   <xacro:macro name="insert_visualization_waist_yaw" params="">
     <visual>
-      <origin xyz="0 0 0.025" rpy="0 0 0"/>
+      <origin xyz="0 0 -0.001" rpy="0 0 0"/>
       <geometry>
-         <!--sphere radius="1.0"/-->
-         <cylinder radius="0.02" length="0.06"/>
+        <mesh filename="package://teo_description/meshes/torso/waist-yaw.stl"/>
       </geometry>
-      <material name="LightGrey"/>
+      <material name="teoGray"/>
     </visual>
     <collision>
@@ -28,10 +24,9 @@
   <xacro:macro name="insert_visualization_waist_pitch" params="">
     <visual>
-      <origin xyz="0 0 0" rpy="${pi_2} 0 0"/>
+      <origin xyz="0 0 0" rpy="0 0 0"/>
       <geometry>
-        <!--sphere radius="1.0"/-->
-        <cylinder radius="0.02" length="0.06"/>
+        <mesh filename="package://teo_description/meshes/torso/waist-pitch.stl"/>
       </geometry>
-      <material name="LightGrey"/>
+      <material name="teoGray"/>
     </visual>
     <collision>
@@ -45,7 +40,35 @@
   <xacro:macro name="insert_visualization_torso" params="">
     <visual>
-      <origin xyz="-0.005 0 0.065" rpy="0 0 0"/>
+      <origin xyz="0 0 ${torso_link2}" rpy="0 0 0"/>
       <geometry>
-        <mesh filename="package://teo_description/meshes/torso/chest_reduced2.dae"/>
+        <mesh filename="package://teo_description/meshes/torso/torso.stl"/>
+      </geometry>
+      <material name="teoGray"/>
+    </visual>
+    <visual>
+      <origin xyz="0 0.25486 ${torso_link2+chest_link2}" rpy="0 0 0"/>
+      <geometry>
+        <mesh filename="package://teo_description/meshes/torso/L-torso-shoulder.stl"/>
+      </geometry>
+      <material name="teoGray"/>
+    </visual>
+    <visual>
+      <origin xyz="0 -0.25486 ${torso_link2+chest_link2}" rpy="0 0 0"/>
+      <geometry>
+        <mesh filename="package://teo_description/meshes/torso/R-torso-shoulder.stl"/>
+      </geometry>
+      <material name="LightGrey"/>
+    </visual>
+    <visual>
+      <origin xyz="0 0 0.346" rpy="0 0 0"/>
+      <geometry>
+        <mesh filename="package://teo_description/meshes/torso/neck.stl"/>
+      </geometry>
+      <material name="LightGrey"/>
+    </visual>
+    <visual>
+      <origin xyz="0 0 0.434" rpy="0 0 0"/>
+      <geometry>
+        <mesh filename="package://teo_description/meshes/torso/head.stl"/>
       </geometry>
       <material name="LightGrey"/>
@@ -59,11 +82,18 @@
   </xacro:macro>
   <xacro:macro name="insert_visualization_waist" params="">
-    <!--visual>
+    <visual>
+      <origin xyz="0 0 0" rpy="0 0 0"/>
       <geometry>
-        <mesh filename="package://teo_description/meshes/torso/waist.dae"/>
+        <mesh filename="package://teo_description/meshes/torso/waist-base.stl"/>
       </geometry>
-      <material name="grey"/>
-      <origin rpy="0 0 0" xyz="0 0 0.05"/>
-    </visual-->
+      <material name="teoBlack"/>
+    </visual>
+    <visual>
+      <origin xyz="0 0 0.07336" rpy="0 0 0"/>
+      <geometry>
+        <mesh filename="package://teo_description/meshes/torso/waist-link.stl"/>
+      </geometry>
+      <material name="teoGray"/>
+    </visual>
   </xacro:macro>
 </robot>
