Commit message: changing teo_gazebo launch process

File: teo_description/urdf/arms/arm.urdf.xacro (robot description, xacro)
@@ -135,5 +135,5 @@
   </xacro:macro>
   <!-- Joints -->
-  <xacro:macro name="arms_joints" params="side reflect">
+  <xacro:macro name="arms_joints" params="side reflect effortTransmission velocityTransmission positionTransmission">
     <joint name="${side}_shoulder_pitch" type="revolute">
       <parent link="waist_pitch_link"/>
@@ -178,14 +178,14 @@
       <limit velocity="${wrist_pitch_velocity}" effort="${wrist_pitch_effort}" lower="${wrist_pitch_lower}" upper="${wrist_pitch_upper}"/>
     </joint>
-    <xacro:limb_joint_simple_transmission name="shoulder" side="${side}" axis="pitch" reduction="${shoulder_pitch_reduction}"/>
-    <xacro:limb_joint_simple_transmission name="shoulder" side="${side}" axis="roll" reduction="${shoulder_roll_reduction}"/>
-    <xacro:limb_joint_simple_transmission name="shoulder" side="${side}" axis="yaw" reduction="${shoulder_yaw_reduction}"/>
-    <xacro:limb_joint_simple_transmission name="elbow" side="${side}" axis="pitch" reduction="${elbow_pitch_reduction}"/>
-    <xacro:limb_joint_simple_transmission name="wrist" side="${side}" axis="yaw" reduction="${wrist_yaw_reduction}"/>
-    <xacro:limb_joint_simple_transmission name="wrist" side="${side}" axis="pitch" reduction="${wrist_pitch_reduction}"/>
+    <xacro:limb_joint_simple_transmission name="shoulder" side="${side}" axis="pitch" reduction="${shoulder_pitch_reduction}" effortTransmission="${effortTransmission}" velocityTransmission="${velocityTransmission}" positionTransmission="${positionTransmission}"/>
+    <xacro:limb_joint_simple_transmission name="shoulder" side="${side}" axis="roll" reduction="${shoulder_roll_reduction}" effortTransmission="${effortTransmission}" velocityTransmission="${velocityTransmission}" positionTransmission="${positionTransmission}"/>
+    <xacro:limb_joint_simple_transmission name="shoulder" side="${side}" axis="yaw" reduction="${shoulder_yaw_reduction}" effortTransmission="${effortTransmission}" velocityTransmission="${velocityTransmission}" positionTransmission="${positionTransmission}"/>
+    <xacro:limb_joint_simple_transmission name="elbow" side="${side}" axis="pitch" reduction="${elbow_pitch_reduction}" effortTransmission="${effortTransmission}" velocityTransmission="${velocityTransmission}" positionTransmission="${positionTransmission}"/>
+    <xacro:limb_joint_simple_transmission name="wrist" side="${side}" axis="yaw" reduction="${wrist_yaw_reduction}" effortTransmission="${effortTransmission}" velocityTransmission="${velocityTransmission}" positionTransmission="${positionTransmission}"/>
+    <xacro:limb_joint_simple_transmission name="wrist" side="${side}" axis="pitch" reduction="${wrist_pitch_reduction}" effortTransmission="${effortTransmission}" velocityTransmission="${velocityTransmission}" positionTransmission="${positionTransmission}"/>
   </xacro:macro>
   <xacro:arms_links side="l" reflect="1"/>
   <xacro:arms_links side="r" reflect="-1"/>
-  <xacro:arms_joints side="l" reflect="1"/>
-  <xacro:arms_joints side="r" reflect="-1"/>
+  <xacro:arms_joints side="l" reflect="1" effortTransmission="1" velocityTransmission="0" positionTransmission="0"/>
+  <xacro:arms_joints side="r" reflect="-1" effortTransmission="1" velocityTransmission="0" positionTransmission="0"/>
 </robot>

File: teo_description/urdf/legs/leg.urdf.xacro (robot description, xacro)
@@ -72,8 +72,5 @@
         <origin xyz="0.0 ${reflect*0.0} 0.0" rpy="0 0 0"/>
         <mass value="0.001"/>
-        <inertia
-				  ixx="0.001" ixy="0.000" ixz="0.000"
-					iyy="0.001" iyz="0.000"
-					izz="0.001" />
+        <inertia ixx="0.00132187534" ixy="0.00000001514" ixz="0.00040022268" iyy="0.0018528617" iyz="0.00000050713" izz="0.00084231334"/>
       </inertial>
 			<xacro:insert_visualization_hip_yaw side="${side}" reflect="{reflect}"/>
@@ -83,8 +80,5 @@
         <origin xyz="-0.029398 ${reflect*0.001062} -0.017753" rpy="0 0 0"/>
         <mass value="0.001"/>
-        <inertia
-				  ixx="0.000001" ixy="0.00000" ixz="0.00000"
-				  iyy="0.000002" iyz="0.00000"
-					izz="0.000001" />
+        <inertia ixx="0.0008416476" ixy="-0.00000268743" ixz="0.00000667199" iyy="0.00039794844" iyz="0.00002668971" izz="0.00084196694"/>
       </inertial>
 			<xacro:insert_visualization_hip_pitch side="${side}" reflect="{reflect}"/>
@@ -94,8 +88,5 @@
         <origin xyz="${0.013-0.008362} ${reflect*0.000115} ${-leg_link2+0.167156}" rpy="0 0 0"/>
         <mass value="1.844"/>
-        <inertia
-				  ixx="0.000020" ixy="0.000000" ixz="0.000000"
-					iyy="0.000018" iyz="0.000002"
-					izz="0.000005" />
+        <inertia ixx="0.00507885174" ixy="-0.00034076421" ixz="-0.00225952731" iyy="0.02850097402" iyz="0.00003047874" izz="0.02632392239"/>
       </inertial>
       <xacro:insert_visualization_femur_link side="${side}" reflect="${reflect}"/>
@@ -105,8 +96,5 @@
         <origin xyz="${-0.013-0.001019} ${reflect*(-(leg_link4)+0.024670)} ${-leg_link3+0.127850}" rpy="0 0 0"/>
         <mass value="2.0817"/>
-        <inertia
-          ixx="0.000011" ixy="0.000000" ixz="0.000000"
-          iyy="0.000010" iyz="0.000000"
-          izz="0.000003" />
+        <inertia ixx="0.00361006492" ixy="0.00012218208" ixz="0.00160208242" iyy="0.02470649045" iyz="0.00008129755" izz="0.02272322206"/>
       </inertial>
       <xacro:insert_visualization_tibia_link side="${side}" reflect="${reflect}"/>
@@ -116,8 +104,5 @@
         <origin xyz="0.004952 ${reflect*-0.005263} 0.028198" rpy="0 0 0"/>
         <mass value="1.0"/>
-        <inertia
-				  ixx="0.000001" ixy="0.000000" ixz="0.000000"
-					iyy="0.000001" iyz="0.000000"
-					izz="0.000001" />
+        <inertia ixx="0.00082035023" ixy="0.00000048534" ixz="0.00000226301" iyy="0.00082074105" iyz="-0.00002892247" izz="0.00037614067"/>
       </inertial>
       <xacro:insert_visualization_ankle_pitch side="${side}" reflect="${reflect}"/>
@@ -127,8 +112,5 @@
         <origin xyz="0.018179 ${reflect*0.003551} -0.075080" rpy="0 0 0"/>
         <mass value="3.8994"/>
-        <inertia
-          ixx="0.000003" ixy="0.000000" ixz="0.000001"
-          iyy="0.000006" iyz="0.000000"
-          izz="0.000006" />
+        <inertia ixx="0.00366502559" ixy="0.00020479295" ixz="0.00112439297" iyy="0.00532618026" iyz="0.00012133755" izz="0.00353091463"/>
       </inertial>
       <xacro:insert_visualization_ankle_roll side="${side}" reflect="${reflect}"/>
@@ -138,8 +120,5 @@
         <origin xyz="0.0 ${reflect*0.0} 0.0" rpy="0 0 0"/>
         <mass value="0.001"/>
-        <inertia
-				  ixx="0.001" ixy="0.000" ixz="0.000"
-					iyy="0.001" iyz="0.000"
-					izz="0.001" />
+        <inertia ixx="0.0" ixy="0.0" ixz="0.0" iyy="0.0" iyz="0.0" izz="0.0"/>
       </inertial>
       <xacro:insert_visualization_foot side="${side}" reflect="${reflect}"/>
@@ -148,5 +127,5 @@
   </xacro:macro>
   <!-- Joints -->
-  <xacro:macro name="legs_joints" params="side reflect">
+  <xacro:macro name="legs_joints" params="side reflect effortTransmission velocityTransmission positionTransmission">
     <joint name="${side}_hip_yaw" type="revolute">
       <parent link="waist"/>
@@ -202,14 +181,14 @@
       <origin xyz="0 0 -${leg_link5}" rpy="0 0 0"/>
     </joint>
-    <xacro:limb_joint_simple_transmission name="hip" side="${side}" axis="yaw" reduction="${hip_yaw_reduction}"/>
-    <xacro:limb_joint_simple_transmission name="hip" side="${side}" axis="roll" reduction="${hip_roll_reduction}"/>
-    <xacro:limb_joint_simple_transmission name="hip" side="${side}" axis="pitch" reduction="${hip_pitch_reduction}"/>
-    <xacro:limb_joint_simple_transmission name="knee" side="${side}" axis="pitch" reduction="${knee_pitch_reduction}"/>
-    <xacro:limb_joint_simple_transmission name="ankle" side="${side}" axis="pitch" reduction="${ankle_pitch_reduction}"/>
-    <xacro:limb_joint_simple_transmission name="ankle" side="${side}" axis="roll" reduction="${ankle_roll_reduction}"/>
+    <xacro:limb_joint_simple_transmission name="hip" side="${side}" axis="yaw" reduction="${hip_yaw_reduction}" effortTransmission="${effortTransmission}" velocityTransmission="${velocityTransmission}" positionTransmission="${positionTransmission}"/>
+    <xacro:limb_joint_simple_transmission name="hip" side="${side}" axis="roll" reduction="${hip_roll_reduction}" effortTransmission="${effortTransmission}" velocityTransmission="${velocityTransmission}" positionTransmission="${positionTransmission}"/>
+    <xacro:limb_joint_simple_transmission name="hip" side="${side}" axis="pitch" reduction="${hip_pitch_reduction}" effortTransmission="${effortTransmission}" velocityTransmission="${velocityTransmission}" positionTransmission="${positionTransmission}"/>
+    <xacro:limb_joint_simple_transmission name="knee" side="${side}" axis="pitch" reduction="${knee_pitch_reduction}" effortTransmission="${effortTransmission}" velocityTransmission="${velocityTransmission}" positionTransmission="${positionTransmission}"/>
+    <xacro:limb_joint_simple_transmission name="ankle" side="${side}" axis="pitch" reduction="${ankle_pitch_reduction}" effortTransmission="${effortTransmission}" velocityTransmission="${velocityTransmission}" positionTransmission="${positionTransmission}"/>
+    <xacro:limb_joint_simple_transmission name="ankle" side="${side}" axis="roll" reduction="${ankle_roll_reduction}" effortTransmission="${effortTransmission}" velocityTransmission="${velocityTransmission}" positionTransmission="${positionTransmission}"/>
   </xacro:macro>
   <xacro:legs_links side="l" reflect="1"/>
   <xacro:legs_links side="r" reflect="-1"/>
-  <xacro:legs_joints side="l" reflect="1"/>
-  <xacro:legs_joints side="r" reflect="-1"/>
+  <xacro:legs_joints side="l" reflect="1" effortTransmission="0" velocityTransmission="0" positionTransmission="1"/>
+  <xacro:legs_joints side="r" reflect="-1" effortTransmission="0" velocityTransmission="0" positionTransmission="1"/>
 </robot>

File: teo_description/urdf/others/teo_transmission.xacro (robot description, xacro)
@@ -5,14 +5,41 @@
 -->
 <robot name="teo" xmlns:xacro="http://ros.org/wiki/xacro">
-	<xacro:macro name="limb_joint_simple_transmission" params="name side axis reduction" >
-		<transmission name="${side}_${name}_${axis}_trans">
-			<type>transmission_interface/SimpleTransmission</type>
-			<joint name="${side}_${name}_${axis}">
-				<hardwareInterface>EffortJointInterface</hardwareInterface>
-      </joint>
-			<actuator name="${side}_${name}_${axis}_motor" >
-				<mechanicalReduction>${reduction}</mechanicalReduction>
-			</actuator>
-		</transmission>
+	<xacro:macro name="limb_joint_simple_transmission" params="name side axis reduction effortTransmission velocityTransmission positionTransmission" >
+		<xacro:if value="${effortTransmission}">
+			<transmission name="${side}_${name}_${axis}_trans">
+				<type>transmission_interface/SimpleTransmission</type>
+				<joint name="${side}_${name}_${axis}">
+					<hardwareInterface>EffortJointInterface</hardwareInterface>
+	      </joint>
+				<actuator name="${side}_${name}_${axis}_motor" >
+					<hardwareInterface>EffortJointInterface</hardwareInterface>
+					<mechanicalReduction>${reduction}</mechanicalReduction>
+				</actuator>
+			</transmission>
+    </xacro:if>
+    <xacro:if value="${velocityTransmission}">
+			<transmission name="${side}_${name}_${axis}_trans">
+				<type>transmission_interface/SimpleTransmission</type>
+				<joint name="${side}_${name}_${axis}">
+					<hardwareInterface>VelocityJointInterface</hardwareInterface>
+	      </joint>
+				<actuator name="${side}_${name}_${axis}_motor" >
+					<hardwareInterface>VelocityJointInterface</hardwareInterface>
+					<mechanicalReduction>${reduction}</mechanicalReduction>
+				</actuator>
+			</transmission>
+    </xacro:if>
+    <xacro:if value="${positionTransmission}">
+			<transmission name="${side}_${name}_${axis}_trans">
+				<type>transmission_interface/SimpleTransmission</type>
+				<joint name="${side}_${name}_${axis}">
+					<hardwareInterface>PositionJointInterface</hardwareInterface>
+	      </joint>
+				<actuator name="${side}_${name}_${axis}_motor" >
+					<hardwareInterface>PositionJointInterface</hardwareInterface>
+					<mechanicalReduction>${reduction}</mechanicalReduction>
+				</actuator>
+			</transmission>
+    </xacro:if>
 	</xacro:macro>
 	<xacro:macro name="waist_joint_simple_transmission" params="axis reduction" >

File: teo_description/urdf/teo_humanoid.gazebo.xacro (robot description, xacro)
@@ -14,16 +14,16 @@
 			<mu1>0.9</mu1>
 			<mu2>0.9</mu2>
-			<material>Gazebo/FlatBlack</material>
+			<material>Gazebo/White</material>
 		</gazebo>
 		<gazebo reference="waist_pitch_link">
 			<mu1>0.9</mu1>
 			<mu2>0.9</mu2>
-			<material>Gazebo/Green</material>
+			<material>Gazebo/White</material>
 		</gazebo>
-		<!--gazebo reference="waist">
+<!-- 		<gazebo reference="waist">
 			<mu1>0.9</mu1>
 			<mu2>0.9</mu2>
-			<material>Gazebo/Red</material>
-		</gazebo-->
+			<material>Gazebo/White</material>
+		</gazebo> -->
 	</xacro:macro>
 	<!-- ############## -->
@@ -34,35 +34,44 @@
 			<mu1>0.9</mu1>
 			<mu2>0.9</mu2>
-			<material>Gazebo/Purple</material>
+			<material>Gazebo/White</material>
 		</gazebo>
 		<gazebo reference="${side}_hip_yaw_link">
 			<mu1>0.9</mu1>
 			<mu2>0.9</mu2>
-			<material>Gazebo/SkyBlue</material>
+			<material>Gazebo/White</material>
 		</gazebo>
 		<gazebo reference="${side}_femur_link">
 			<mu1>0.9</mu1>
 			<mu2>0.9</mu2>
-			<material>Gazebo/Orange</material>
+			<material>Gazebo/White</material>
 		</gazebo>
 		<gazebo reference="${side}_tibia_link">
 			<mu1>0.9</mu1>
 			<mu2>0.9</mu2>
-			<material>Gazebo/Black</material>
+			<material>Gazebo/White</material>
 		</gazebo>
 		<gazebo reference="${side}_ankle_pitch_link">
 			<mu1>0.9</mu1>
 			<mu2>0.9</mu2>
-			<material>Gazebo/Green</material>
+			<material>Gazebo/White</material>
 		</gazebo>
 		<gazebo reference="${side}_astragalus_link">
-			<mu1>0.9</mu1>
-			<mu2>0.9</mu2>
-			<material>Gazebo/Yellow</material>
+			<kp>1000000.0</kp>
+			<kd>100.0</kd>
+			<mu1>1.0</mu1>
+			<mu2>1.0</mu2>
+			<fdir1>0 0 1</fdir1>
+			<maxVel>1.0</maxVel>
+			<minDepth>0.00</minDepth>
+			<implicitSpringDamper>1</implicitSpringDamper>
+			<material>Gazebo/White</material>
 		</gazebo>
 		<gazebo reference="${side}_sole">
-			<mu1>0.9</mu1>
-			<mu2>0.9</mu2>
-			<material>Gazebo/Grey</material>
+	    <mu1>0.9</mu1>
+	    <mu2>0.9</mu2>
+	    <fdir1>1 0 0</fdir1>
+	    <maxVel>1.0</maxVel>
+	    <minDepth>0.003</minDepth>
+	    <material>Gazebo/White</material>
 		</gazebo>
   </xacro:macro>
@@ -74,30 +83,30 @@
 			<mu1>0.9</mu1>
 			<mu2>0.9</mu2>
-			<material>Gazebo/Turquoise</material>
+			<material>Gazebo/White</material>
 		</gazebo>
 		<gazebo reference="${side}_shoulder_roll_link">
 			<mu1>0.9</mu1>
 			<mu2>0.9</mu2>
-			<material>Gazebo/ZincYellow</material>
+			<material>Gazebo/White</material>
 		</gazebo>
 		<gazebo reference="${side}_shoulder_yaw_link">
 			<mu1>0.9</mu1>
 			<mu2>0.9</mu2>
-			<material>Gazebo/Blue</material>
+			<material>Gazebo/White</material>
 		</gazebo>
 		<gazebo reference="${side}_elbow_pitch_link">
 			<mu1>0.9</mu1>
 			<mu2>0.9</mu2>
-			<material>Gazebo/RedBright</material>
+			<material>Gazebo/White</material>
 		</gazebo>
 		<gazebo reference="${side}_wrist_yaw_link">
 			<mu1>0.9</mu1>
 			<mu2>0.9</mu2>
-			<material>Gazebo/SkyBlue</material>
+			<material>Gazebo/White</material>
 		</gazebo>
 		<gazebo reference="${side}_wrist_pitch_link">
 			<mu1>0.9</mu1>
 			<mu2>0.9</mu2>
-			<material>Gazebo/Green</material>
+			<material>Gazebo/White</material>
 		</gazebo>
 	</xacro:macro>

File: teo_description/urdf/teo_humanoid.urdf (robot description, URDF)
Before this commit: robot teo, 30 links, 29 joints
Links:
- link l_ankle_pitch_link: geometry visual mesh filename=package://teo_description/meshes/legs/l_ankle_pitch.stl
- link l_astragalus_link: geometry visual mesh filename=package://teo_description/meshes/legs/l_ankle_roll.stl; visual mesh filename=package://teo_description/meshes/legs/l_ankle_sensorFT.stl
- link l_elbow_pitch_link: geometry collision box size=0.06 0.06 0.202; visual mesh filename=package://teo_description/meshes/arms/l_elbow_link.stl
- link l_femur_link: geometry collision box size=0.1 0.1 0.33; visual mesh filename=package://teo_description/meshes/legs/l_femur.stl
- link l_hip_roll_link: geometry visual mesh filename=package://teo_description/meshes/legs/l_hip_pitch.stl
- link l_hip_yaw_link: geometry collision cylinder length=0.13 radius=0.045; visual mesh filename=package://teo_description/meshes/legs/l_hip_yaw.stl
- link l_shoulder_pitch_link: geometry collision box size=0.1 0.34 0.1; visual mesh filename=package://teo_description/meshes/arms/l_shoulder_pitch.stl
- link l_shoulder_roll_link: geometry collision box size=0.1 0.34 0.1; visual mesh filename=package://teo_description/meshes/arms/l_shoulder_roll.stl
- link l_shoulder_yaw_link: geometry collision box size=0.08 0.08 0.32901; visual mesh filename=package://teo_description/meshes/arms/l_humerus.stl
- link l_sole: geometry collision box size=0.08 0.08 0.124; visual mesh filename=package://teo_description/meshes/legs/l_foot.stl
- link l_tibia_link: geometry collision box size=0.05 0.033 0.05; visual mesh filename=package://teo_description/meshes/legs/l_tibia.stl
- link l_wrist_pitch_link: geometry collision box size=0.03 0.03 0.03; visual mesh filename=package://teo_description/meshes/arms/l_hand.stl
- link l_wrist_yaw_link: geometry collision box size=0.03 0.03 0.03; visual mesh filename=package://teo_description/meshes/arms/l_wrist_yaw.stl
- link r_ankle_pitch_link: geometry visual mesh filename=package://teo_description/meshes/legs/r_ankle_pitch.stl
- link r_astragalus_link: geometry visual mesh filename=package://teo_description/meshes/legs/r_ankle_roll.stl; visual mesh filename=package://teo_description/meshes/legs/r_ankle_sensorFT.stl
- link r_elbow_pitch_link: geometry collision box size=0.06 0.06 0.202; visual mesh filename=package://teo_description/meshes/arms/r_elbow_link.stl
- link r_femur_link: geometry collision box size=0.1 0.1 0.33; visual mesh filename=package://teo_description/meshes/legs/r_femur.stl
- link r_hip_roll_link: geometry visual mesh filename=package://teo_description/meshes/legs/r_hip_pitch.stl
- link r_hip_yaw_link: geometry collision cylinder length=0.13 radius=0.045; visual mesh filename=package://teo_description/meshes/legs/r_hip_yaw.stl
- link r_shoulder_pitch_link: geometry collision box size=0.1 0.34 0.1; visual mesh filename=package://teo_description/meshes/arms/r_shoulder_pitch.stl
- link r_shoulder_roll_link: geometry collision box size=0.1 0.34 0.1; visual mesh filename=package://teo_description/meshes/arms/r_shoulder_roll.stl
- link r_shoulder_yaw_link: geometry collision box size=0.08 0.08 0.32901; visual mesh filename=package://teo_description/meshes/arms/r_humerus.stl
- link r_sole: geometry collision box size=0.08 0.08 0.124; visual mesh filename=package://teo_description/meshes/legs/r_foot.stl
- link r_tibia_link: geometry collision box size=0.05 0.033 0.05; visual mesh filename=package://teo_description/meshes/legs/r_tibia.stl
- link r_wrist_pitch_link: geometry collision box size=0.03 0.03 0.03; visual mesh filename=package://teo_description/meshes/arms/r_hand.stl
- link r_wrist_yaw_link: geometry collision box size=0.03 0.03 0.03; visual mesh filename=package://teo_description/meshes/arms/r_wrist_yaw.stl
- link waist: geometry visual mesh filename=package://teo_description/meshes/torso/waist-base.stl; visual mesh filename=package://teo_description/meshes/torso/waist-link.stl
- link waist_pitch_link: geometry collision box size=0.18 0.42 0.292; collision cylinder length=0.06 radius=0.02
- link waist_yaw_link: geometry collision cylinder length=0.06 radius=0.02; visual mesh filename=package://teo_description/meshes/torso/waist-yaw.stl
Joints:
- joint l_elbow_pitch: origin xyz=0 0 -0.337 rpy=0 0 0 -> xyz=0 0 -0.32901 rpy=0 0 0
- joint l_hip_yaw: origin xyz=0 0.146 0 rpy=0 0 0 -> xyz=0 0.146 -0.10237 rpy=0 0 0
- joint l_shoulder_pitch: origin xyz=-0.0 0.34 0.245 rpy=0 0 0 -> xyz=-0.0 0.34 0.305 rpy=0 0 0
- joint l_wrist_yaw: origin xyz=0 0 -0.21 rpy=0 0 0 -> xyz=0 0 -0.202 rpy=0 0 0
- joint r_elbow_pitch: origin xyz=0 0 -0.337 rpy=0 0 0 -> xyz=0 0 -0.32901 rpy=0 0 0
- joint r_hip_yaw: origin xyz=0 -0.146 0 rpy=0 0 0 -> xyz=0 -0.146 -0.10237 rpy=0 0 0
- joint r_shoulder_pitch: origin xyz=-0.0 -0.34 0.245 rpy=0 0 0 -> xyz=-0.0 -0.34 0.305 rpy=0 0 0
- joint r_wrist_yaw: origin xyz=0 0 -0.21 rpy=0 0 0 -> xyz=0 0 -0.202 rpy=0 0 0
- joint waist_yaw: origin xyz=0.0 0 0.287 rpy=0 0 0 -> xyz=0.0 0 0.1907 rpy=0 0 0
