Commit message: change of the collision of foot in xacro file

File: teo_description/urdf/legs/legs_vis.urdf.xacro (robot description, xacro)
@@ -94,7 +94,8 @@
     <collision>
       <geometry>
-        <box size="0.08 0.08 ${leg_link5}"/>
+        <!-- <box size="0.08 0.08 ${leg_link5}"/> -->
+        <box size="0.245438 0.139979 0.019500"/>
       </geometry>
-      <origin rpy="0 0 0" xyz="0 0 -${leg_link5/2}"/>
+      <origin rpy="0 0 0" xyz="0.05 0 0.00975"/>
     </collision>
   </xacro:macro>
