Commit message: teo_tf package added to the metapackage

File: teo_description/urdf/legs/leg.urdf.xacro (robot description, xacro)
@@ -72,73 +72,73 @@
         <mass value="0.001"/>
         <inertia
-				  ixx="1.000" ixy="0.000" ixz="0.000"
-					iyy="1.000" iyz="0.000"
-					izz="1.000" />
+				  ixx="0.001" ixy="0.000" ixz="0.000"
+					iyy="0.001" iyz="0.000"
+					izz="0.001" />
       </inertial>
     </link>
     <link name="${side}_hip_roll_link">
+      <inertial>
+        <origin xyz="-0.029398 ${reflect*0.001062} -0.017753" rpy="0 0 0"/>
+        <mass value="0.001"/>
+        <inertia
+				  ixx="0.000001" ixy="0.00000" ixz="0.00000"
+				  iyy="0.000002" iyz="0.00000"
+					izz="0.000001" />
+      </inertial>
+			<xacro:insert_visualization_hip_roll side="${side}" reflect="{reflect}"/>
+    </link>
+    <link name="${side}_femur_link">
+      <inertial>
+        <origin xyz="${0.013-0.008362} ${reflect*0.000115} ${-leg_link2+0.167156}" rpy="0 0 0"/>
+        <mass value="1.844"/>
+        <inertia
+				  ixx="0.000020" ixy="0.000000" ixz="0.000000"
+					iyy="0.000018" iyz="0.000002"
+					izz="0.000005" />
+      </inertial>
+      <xacro:insert_visualization_femur_link side="${side}" reflect="${reflect}"/>
+    </link>
+    <link name="${side}_tibia_link">
+      <inertial>
+        <origin xyz="${-0.013-0.001019} ${reflect*(-(leg_link4)+0.024670)} ${-leg_link3+0.127850}" rpy="0 0 0"/>
+        <mass value="2.0817"/>
+        <inertia
+          ixx="0.000011" ixy="0.000000" ixz="0.000000"
+          iyy="0.000010" iyz="0.000000"
+          izz="0.000003" />
+      </inertial>
+      <xacro:insert_visualization_tibia_link side="${side}" reflect="${reflect}"/>
+    </link>
+    <link name="${side}_ankle_pitch_link">
+      <inertial>
+        <origin xyz="0.004952 ${reflect*-0.005263} 0.028198" rpy="0 0 0"/>
+        <mass value="1.0"/>
+        <inertia
+				  ixx="0.000001" ixy="0.000000" ixz="0.000000"
+					iyy="0.000001" iyz="0.000000"
+					izz="0.000001" />
+      </inertial>
+      <xacro:insert_visualization_ankle_pitch side="${side}" reflect="${reflect}"/>
+    </link>
+    <link name="${side}_astragalus_link">
+      <inertial>
+        <origin xyz="0.018179 ${reflect*0.003551} -0.075080" rpy="0 0 0"/>
+        <mass value="3.8994"/>
+        <inertia
+          ixx="0.000003" ixy="0.000000" ixz="0.000001"
+          iyy="0.000006" iyz="0.000000"
+          izz="0.000006" />
+      </inertial>
+      <xacro:insert_visualization_astragalus_link side="${side}" reflect="${reflect}"/>
+      <xacro:insert_visualization_sole side="${side}" reflect="${reflect}"/> <!-- OJO, falta bajarlo -link5/2-->
+    </link>
+    <link name="${side}_sole">
       <inertial>
         <origin xyz="0.0 ${reflect*0.0} 0.0" rpy="0 0 0"/>
         <mass value="0.001"/>
         <inertia
-				  ixx="1.000" ixy="0.000" ixz="0.000"
-				  iyy="1.000" iyz="0.000"
-					izz="1.000" />
-      </inertial>
-			<xacro:insert_visualization_hip_roll side="${side}" reflect="{reflect}"/>
-    </link>
-    <link name="${side}_femur_link">
-      <inertial>
-        <origin xyz="0.033 ${reflect*leg_link4+0.001} ${leg_link3+leg_link2-0.443}" rpy="0 0 0"/>
-        <mass value="1.844"/>
-        <inertia
-				  ixx="0.020" ixy="6.052e-5" ixz="7.948e-4"
-					iyy="0.025" iyz="6.454e-4"
-					izz="0.013" />
-      </inertial>
-      <xacro:insert_visualization_femur_link side="${side}" reflect="${reflect}"/>
-    </link>
-    <link name="${side}_tibia_link">
-      <inertial>
-        <origin xyz="-0.027 ${reflect*leg_link4-0.005} ${leg_link3-0.16368}" rpy="0 0 0"/>
-        <mass value="2.0817"/>
-        <inertia
-				  ixx="0.020" ixy="6.052e-5" ixz="-7.498e-4"
-				  iyy="0.025" iyz="6.454e-4"
-					izz="0.013" />
-      </inertial>
-      <xacro:insert_visualization_tibia_link side="${side}" reflect="${reflect}"/>
-    </link>
-    <link name="${side}_ankle_pitch_link">
-      <inertial>
-        <origin xyz="0.0 ${reflect*0.0} 0.0" rpy="0 0 0"/>
-        <mass value="1.0"/>
-        <inertia
-				  ixx="1.000" ixy="0.000" ixz="0.000"
-					iyy="1.000" iyz="0.000"
-					izz="1.000" />
-      </inertial>
-      <xacro:insert_visualization_ankle_pitch side="${side}" reflect="${reflect}"/>
-    </link>
-    <link name="${side}_astragalus_link">
-      <inertial>
-        <origin xyz="3.026e-3 ${reflect*3.5e-3} -9.323e-3" rpy="0 0 0"/>
-        <mass value="3.8994"/>
-        <inertia
-				  ixx="0.062" ixy="-1.417e-4" ixz="-0.004"
-					iyy="0.059" iyz="0.002"
-					izz="0.011" />
-      </inertial>
-      <xacro:insert_visualization_astragalus_link side="${side}" reflect="${reflect}"/>
-      <xacro:insert_visualization_sole side="${side}" reflect="${reflect}"/> <!-- OJO, falta bajarlo -link5/2-->
-    </link>
-    <link name="${side}_sole">
-      <inertial>
-        <origin xyz="0.0 ${reflect*0.0} 0.0" rpy="0 0 0"/>
-        <mass value="0.001"/>
-        <inertia
-				  ixx="1.000" ixy="0.000" ixz="0.000"
-					iyy="1.000" iyz="0.000"
-					izz="1.000" />
+				  ixx="0.001" ixy="0.000" ixz="0.000"
+					iyy="0.001" iyz="0.000"
+					izz="0.001" />
       </inertial>
     </link>

Commit message: changing joints controller 1

File: teo_description/urdf/legs/leg.urdf.xacro (robot description, xacro)
@@ -31,31 +31,31 @@
 	<xacro:property name="ankle_roll_upper" value="${85 * deg_to_rad}" />
 <!-- Effort limit of the angles -->
-	<xacro:property name="hip_yaw_effort" value="30.0" />
-	<xacro:property name="hip_roll_effort" value="30.0" />
-	<xacro:property name="hip_pitch_effort" value="30.0" />
-	<xacro:property name="knee_pitch_effort" value="30.0" />
-	<xacro:property name="ankle_pitch_effort" value="30.0" />
-	<xacro:property name="ankle_roll_effort" value="30.0" />
+	<xacro:property name="hip_yaw_effort" value="45.0" />
+	<xacro:property name="hip_roll_effort" value="65.0" />
+	<xacro:property name="hip_pitch_effort" value="60.0" />
+	<xacro:property name="knee_pitch_effort" value="140.0" />
+	<xacro:property name="ankle_pitch_effort" value="85.0" />
+	<xacro:property name="ankle_roll_effort" value="65.0" />
 <!-- Velocity limit of the angles-->
-	<xacro:property name="hip_yaw_velocity" value="3.0" />
-	<xacro:property name="hip_roll_velocity" value="3.0" />
-	<xacro:property name="hip_pitch_velocity" value="3.0" />
-	<xacro:property name="knee_pitch_velocity" value="3.0" />
-	<xacro:property name="ankle_pitch_velocity" value="3.0" />
-	<xacro:property name="ankle_roll_velocity" value="3.0" />
+	<xacro:property name="hip_yaw_velocity" value="4.0" />
+	<xacro:property name="hip_roll_velocity" value="4.0" />
+	<xacro:property name="hip_pitch_velocity" value="4.0" />
+	<xacro:property name="knee_pitch_velocity" value="4.0" />
+	<xacro:property name="ankle_pitch_velocity" value="4.0" />
+	<xacro:property name="ankle_roll_velocity" value="4.0" />
 <!-- Damping of the joints-->
-	<xacro:property name="hip_yaw_damping" value="0.0" />
-	<xacro:property name="hip_roll_damping" value="0.0" />
-	<xacro:property name="hip_pitch_damping" value="0.0" />
-	<xacro:property name="knee_pitch_damping" value="0.0" />
-	<xacro:property name="ankle_pitch_damping" value="0.0" />
-	<xacro:property name="ankle_roll_damping" value="0.0" />
+	<xacro:property name="hip_yaw_damping" value="1.0" />
+	<xacro:property name="hip_roll_damping" value="1.0" />
+	<xacro:property name="hip_pitch_damping" value="1.0" />
+	<xacro:property name="knee_pitch_damping" value="1.0" />
+	<xacro:property name="ankle_pitch_damping" value="1.0" />
+	<xacro:property name="ankle_roll_damping" value="1.0" />
 <!-- Friction of the joints--> <!-- IT'S NOT USED IN GAZEBO-->
-	<xacro:property name="hip_yaw_friction" value="0.0" />
-	<xacro:property name="hip_roll_friction" value="0.0" />
-	<xacro:property name="hip_pitch_friction" value="0.0" />
-	<xacro:property name="knee_pitch_friction" value="0.0" />
-	<xacro:property name="ankle_pitch_friction" value="0.0" />
-	<xacro:property name="ankle_roll_friction" value="0.0" />
+	<xacro:property name="hip_yaw_friction" value="1.0" />
+	<xacro:property name="hip_roll_friction" value="1.0" />
+	<xacro:property name="hip_pitch_friction" value="1.0" />
+	<xacro:property name="knee_pitch_friction" value="1.0" />
+	<xacro:property name="ankle_pitch_friction" value="1.0" />
+	<xacro:property name="ankle_roll_friction" value="1.0" />
 <!-- Joint reductions-->
 	<xacro:property name="hip_yaw_reduction" value="1.0" />
@@ -190,5 +190,5 @@
   <xacro:legs_links side="l" reflect="1"/>
   <xacro:legs_links side="r" reflect="-1"/>
-  <xacro:legs_joints side="l" reflect="1" effortTransmission="0" velocityTransmission="0" positionTransmission="1"/>
-  <xacro:legs_joints side="r" reflect="-1" effortTransmission="0" velocityTransmission="0" positionTransmission="1"/>
+  <xacro:legs_joints side="l" reflect="1" effortTransmission="1" velocityTransmission="0" positionTransmission="0"/>
+  <xacro:legs_joints side="r" reflect="-1" effortTransmission="1" velocityTransmission="0" positionTransmission="0"/>
 </robot>

File: teo_description/urdf/torso/torso.urdf.xacro (robot description, xacro)
@@ -44,5 +44,5 @@
     <inertial>
       <origin xyz="0.0 0.0 0.0337" rpy="0 0 0"/>
-      <mass value="25.7044"/>
+      <mass value="5.7044"/>
       <inertia
 			  ixx="0.019" ixy="0.000" ixz="0.000"
@@ -57,7 +57,7 @@
       <mass value="0.1"/>
       <inertia
-			  ixx="1.000" ixy="0.000" ixz="0.000"
-				iyy="1.000" iyz="0.000"
-				izz="1.000" />
+			  ixx="0.1000" ixy="0.000" ixz="0.000"
+				iyy="0.1000" iyz="0.000"
+				izz="0.1000" />
     </inertial>
     <xacro:insert_visualization_waist_yaw/>
@@ -66,9 +66,9 @@
     <inertial>
       <origin xyz="0 0 0" rpy="0 0 0"/>
-      <mass value="1.0"/>
+      <mass value="20.0"/>
       <inertia
-			  ixx="1.000" ixy="0.000" ixz="0.000"
-				iyy="1.000" iyz="0.000"
-				izz="1.000" />
+        ixx="0.34286" ixy="0.000016480" ixz="-0.0012113"
+        iyy="0.12925" iyz="0.000093038"
+        izz="0.26900" />
     </inertial>
     <xacro:insert_visualization_waist_pitch/>

Commit message: new intertia tensors in teo's legs

File: teo_description/urdf/legs/leg.urdf.xacro (robot description, xacro)
@@ -9,4 +9,7 @@
 <robot name="teo" xmlns:xacro="http://ros.org/wiki/xacro">
 <!-- *** TEO LEG PARAMETERS -->
+  <xacro:property name="prop_kg_motor_vol_unit" value="6229.073482" /> <!-- Relation Kg - Volume Unit -->
+  <xacro:property name="prop_kg_femur_vol_unit" value="330.0519062" /> <!-- Relation Kg - Volume Unit -->
+  <xacro:property name="prop_kg_tibia_vol_unit" value="2638.403042" /> <!-- Relation Kg - Volume Unit -->
 <!-- Link lengths -->
 	<xacro:property name="leg_link0" value="0.10237" /> <!-- Hip -->
@@ -70,7 +73,8 @@
     <link name="${side}_hip_yaw_link">
       <inertial>
-        <origin xyz="0.0 ${reflect*0.0} 0.0" rpy="0 0 0"/>
-        <mass value="0.001"/>
-        <inertia ixx="0.00132187534" ixy="0.00000001514" ixz="0.00040022268" iyy="0.0018528617" iyz="0.00000050713" izz="0.00084231334"/>
+        <origin xyz="0.0 ${-reflect*0.0} 0.0" rpy="0 0 0"/>
+        <!-- <mass value="0.001"/> -->
+        <mass value="${prop_kg_motor_vol_unit*0.000185}"/>
+        <inertia ixx="0.00132187534" ixy="${-reflect*0.00000001514}" ixz="0.00040022268" iyy="0.0018528617" iyz="${-reflect*0.00000050713}" izz="0.00084231334"/>
       </inertial>
 			<xacro:insert_visualization_hip_yaw side="${side}" reflect="{reflect}"/>
@@ -78,7 +82,8 @@
     <link name="${side}_hip_roll_link">
       <inertial>
-        <origin xyz="-0.029398 ${reflect*0.001062} -0.017753" rpy="0 0 0"/>
-        <mass value="0.001"/>
-        <inertia ixx="0.0008416476" ixy="-0.00000268743" ixz="0.00000667199" iyy="0.00039794844" iyz="0.00002668971" izz="0.00084196694"/>
+        <origin xyz="-0.029398 ${-reflect*0.001062} -0.017753" rpy="0 0 0"/>
+        <!-- <mass value="0.001"/> -->
+        <mass value="${prop_kg_motor_vol_unit*0.000317}"/>
+        <inertia ixx="0.0008416476" ixy="${-reflect*-0.00000268743}" ixz="0.00000667199" iyy="0.00039794844" iyz="${-reflect*0.00002668971}" izz="0.00084196694"/>
       </inertial>
 			<xacro:insert_visualization_hip_pitch side="${side}" reflect="{reflect}"/>
@@ -86,7 +91,8 @@
     <link name="${side}_femur_link">
       <inertial>
-        <origin xyz="${0.013-0.008362} ${reflect*0.000115} ${-leg_link2+0.167156}" rpy="0 0 0"/>
-        <mass value="1.844"/>
-        <inertia ixx="0.00507885174" ixy="-0.00034076421" ixz="-0.00225952731" iyy="0.02850097402" iyz="0.00003047874" izz="0.02632392239"/>
+        <origin xyz="${0.013-0.008362} ${-reflect*0.000115} ${-leg_link2+0.167156}" rpy="0 0 0"/>
+        <!-- <mass value="1.844"/> -->
+        <mass value="${prop_kg_femur_vol_unit*0.005587}"/>
+        <inertia ixx="0.00507885174" ixy="${-reflect*-0.00034076421}" ixz="-0.00225952731" iyy="0.02850097402" iyz="${-reflect*0.00003047874}" izz="0.02632392239"/>
       </inertial>
       <xacro:insert_visualization_femur_link side="${side}" reflect="${reflect}"/>
@@ -94,7 +100,8 @@
     <link name="${side}_tibia_link">
       <inertial>
-        <origin xyz="${-0.013-0.001019} ${reflect*(-(leg_link4)+0.024670)} ${-leg_link3+0.127850}" rpy="0 0 0"/>
-        <mass value="2.0817"/>
-        <inertia ixx="0.00361006492" ixy="0.00012218208" ixz="0.00160208242" iyy="0.02470649045" iyz="0.00008129755" izz="0.02272322206"/>
+        <origin xyz="${-0.013-0.001019} ${-reflect*(-(leg_link4)+0.024670)} ${-leg_link3+0.127850}" rpy="0 0 0"/>
+        <!-- <mass value="2.0817"/> -->
+        <mass value="${prop_kg_femur_vol_unit*0.005587}"/>
+        <inertia ixx="0.00361006492" ixy="${-reflect*0.00012218208}" ixz="0.00160208242" iyy="0.02470649045" iyz="${-reflect*0.00008129755}" izz="0.02272322206"/>
       </inertial>
       <xacro:insert_visualization_tibia_link side="${side}" reflect="${reflect}"/>
@@ -102,7 +109,7 @@
     <link name="${side}_ankle_pitch_link">
       <inertial>
-        <origin xyz="0.004952 ${reflect*-0.005263} 0.028198" rpy="0 0 0"/>
+        <origin xyz="0.004952 ${-reflect*-0.005263} 0.028198" rpy="0 0 0"/>
         <mass value="1.0"/>
-        <inertia ixx="0.00082035023" ixy="0.00000048534" ixz="0.00000226301" iyy="0.00082074105" iyz="-0.00002892247" izz="0.00037614067"/>
+        <inertia ixx="0.00082035023" ixy="${-reflect*0.00000048534}" ixz="0.00000226301" iyy="0.00082074105" iyz="${-reflect*-0.00002892247}" izz="0.00037614067"/>
       </inertial>
       <xacro:insert_visualization_ankle_pitch side="${side}" reflect="${reflect}"/>
@@ -110,7 +117,7 @@
     <link name="${side}_astragalus_link">
       <inertial>
-        <origin xyz="0.018179 ${reflect*0.003551} -0.075080" rpy="0 0 0"/>
-        <mass value="3.8994"/>
-        <inertia ixx="0.00366502559" ixy="0.00020479295" ixz="0.00112439297" iyy="0.00532618026" iyz="0.00012133755" izz="0.00353091463"/>
+        <origin xyz="-0.006788 ${-reflect*0.000020} -0.042127" rpy="0 0 0"/>
+        <mass value="1.015338978"/>
+        <inertia ixx="0.00026324" ixy="${-reflect*0.0}" ixz="0.0000074" iyy="0.000571" iyz="${-reflect*0}" izz="0.0004633"/>
       </inertial>
       <xacro:insert_visualization_ankle_roll side="${side}" reflect="${reflect}"/>
@@ -118,7 +125,7 @@
     <link name="${side}_sole">
       <inertial>
-        <origin xyz="0.0 ${reflect*0.0} 0.0" rpy="0 0 0"/>
-        <mass value="0.001"/>
-        <inertia ixx="0.0" ixy="0.0" ixz="0.0" iyy="0.0" iyz="0.0" izz="0.0"/>
+        <origin xyz="0.022629 ${-reflect*0.002448} 0.011325" rpy="0 0 0"/>
+        <mass value="2.884061022"/>
+        <inertia ixx="0.006699" ixy="${-reflect*-0.00009295}" ixz="0.00009066" iyy="0.00169929" iyz="${-reflect*0.00000708}" izz="0.00228359"/>
       </inertial>
       <xacro:insert_visualization_foot side="${side}" reflect="${reflect}"/>
