Commit message: inertia matrix in torso

File: teo_description/urdf/legs/leg.urdf.xacro (robot description, xacro)
@@ -75,6 +75,7 @@
         <origin xyz="0.0 ${-reflect*0.0} 0.0" rpy="0 0 0"/>
         <!-- <mass value="0.001"/> -->
-        <mass value="${prop_kg_motor_vol_unit*0.000185}"/>
-        <inertia ixx="3.4076e-7" ixy="${-reflect*0.0}" ixz="5.4e-10" iyy="5.7638e-7" iyz="${-reflect*3.7186e-7}" izz="0.00084231334"/>
+        <mass value="1.0"/>
+        <!-- <mass value="${prop_kg_motor_vol_unit*0.000185}"/> -->
+        <inertia ixx="3.4076E-4" ixy="${-reflect*0.0}" ixz="5.4E-7" iyy="5.7638E-4" iyz="${-reflect*3.7186E-4}" izz="0.84231334"/>
       </inertial>
 			<xacro:insert_visualization_hip_yaw side="${side}" reflect="{reflect}"/>
@@ -82,8 +83,10 @@
     <link name="${side}_hip_roll_link">
       <inertial>
-        <origin xyz="-0.029398 ${-reflect*0.001062} -0.017753" rpy="0 0 0"/>
+        <origin xyz="0.0 ${-reflect*0.0} -0.017753" rpy="0 0 0"/>
+        <!-- <origin xyz="-0.029398 ${-reflect*0.001062} -0.017753" rpy="0 0 0"/> -->
         <!-- <mass value="0.001"/> -->
-        <mass value="${prop_kg_motor_vol_unit*0.000317}"/>
-        <inertia ixx="0.0008416476" ixy="${-reflect*-0.00000268743}" ixz="0.00000667199" iyy="0.00039794844" iyz="${-reflect*0.00002668971}" izz="0.00084196694"/>
+        <mass value="1.0"/>
+        <!-- <mass value="${prop_kg_motor_vol_unit*0.000317}"/> -->
+        <inertia ixx="3.6847E-4" ixy="${-reflect*4.34E-6}" ixz="1.0E-8" iyy="1.9052E-4" iyz="${-reflect*0.0}" izz="4.5536E-4"/>
       </inertial>
 			<xacro:insert_visualization_hip_pitch side="${side}" reflect="{reflect}"/>
@@ -91,8 +94,11 @@
     <link name="${side}_femur_link">
       <inertial>
-        <origin xyz="${-0.013877} ${-reflect*0.0} ${-0.172570}" rpy="0 0 0"/>
+        <origin xyz="0.0 ${-reflect*0.0} ${-0.172570}" rpy="0 0 0"/>
+        <!-- <origin xyz="${-0.013877} ${-reflect*0.0} ${-0.172570}" rpy="0 0 0"/> -->
         <!-- <mass value="1.844"/> -->
-        <mass value="${prop_kg_femur_vol_unit*0.005587}"/>
-        <inertia ixx="0.04453648" ixy="${-reflect*-0.00000001}" ixz="0.00130498" iyy="0.0446349" iyz="${-reflect*0.00000003}" izz="0.02207083"/>
+        <mass value="1.0"/>
+        <!-- <mass value="${prop_kg_femur_vol_unit*0.005587}"/> -->
+        <inertia ixx="4.453648E-2" ixy="${-reflect*-1.0E-8}" ixz="0.00130498" iyy="4.46349E-2" iyz="${-reflect*3.0E-8}" izz="2.207083E-2"/>
+        <!-- <inertia ixx="4.453648E-5" ixy="${-reflect*-1.0E-11}" ixz="0.00000130498" iyy="4.46349E-5" iyz="${-reflect*3.0E-11}" izz="2.207083E-5"/> -->
       </inertial>
       <xacro:insert_visualization_femur_link side="${side}" reflect="${reflect}"/>
@@ -101,8 +107,10 @@
       <inertial>
         <!-- <origin xyz="${-0.013-0.001019} ${-reflect*(-(leg_link4)+0.024670)} ${-leg_link3+0.127850}" rpy="0 0 0"/> -->
-        <origin xyz="${-0.010351} ${-reflect*0.0} -0.142721" rpy="0 0 0"/>
+        <origin xyz="0.0 ${-reflect*0.0} -0.142721" rpy="0 0 0"/>
+        <!-- <origin xyz="${-0.010351} ${-reflect*0.0} -0.142721" rpy="0 0 0"/> -->
         <!-- <mass value="2.0817"/> -->
-        <mass value="${prop_kg_femur_vol_unit*0.005587}"/>
-        <inertia ixx="0.04644211" ixy="${-reflect*0.0}" ixz="-0.00000732" iyy="0.04548272" iyz="${-reflect*0.00000002}" izz="0.00816616"/>
+        <mass value="1.0"/>
+        <!-- <mass value="${prop_kg_femur_vol_unit*0.005587}"/> -->
+        <inertia ixx="4.644211E-2" ixy="${-reflect*0.0}" ixz="-7.32E-6" iyy="4.548272E-2" iyz="${-reflect*-2.0E-8}" izz="8.16616E-3"/>
       </inertial>
       <xacro:insert_visualization_tibia_link side="${side}" reflect="${reflect}"/>
@@ -110,7 +118,11 @@
     <link name="${side}_ankle_pitch_link">
       <inertial>
-        <origin xyz="0.004952 ${-reflect*-0.005263} 0.028198" rpy="0 0 0"/>
-        <mass value="1.0"/>
+        <origin xyz="0.0 ${-reflect*0.0} 0.028198" rpy="0 0 0"/>
+        <!-- <origin xyz="0.004952 ${-reflect*-0.005263} 0.028198" rpy="0 0 0"/> -->
+        <mass value="1.0"/>
+        <!-- <mass value="1.0"/> -->
         <inertia ixx="0.00082035023" ixy="${-reflect*0.00000048534}" ixz="0.00000226301" iyy="0.00082074105" iyz="${-reflect*-0.00002892247}" izz="0.00037614067"/>
+        <!-- REVISAR ESTE!! que falla -->
+        <!-- <inertia ixx="3.3782E-7" ixy="${-reflect*-1.65E-9}" ixz="0.0" iyy="3.8475E-7" iyz="${-reflect*0.0}" izz="5.8551E-7"/> -->
       </inertial>
       <xacro:insert_visualization_ankle_pitch side="${side}" reflect="${reflect}"/>
@@ -118,7 +130,11 @@
     <link name="${side}_astragalus_link">
       <inertial>
-        <origin xyz="-0.006788 ${-reflect*0.000020} -0.042127" rpy="0 0 0"/>
-        <mass value="1.015338978"/>
-        <inertia ixx="0.00026324" ixy="${-reflect*0.0}" ixz="0.0000074" iyy="0.000571" iyz="${-reflect*0}" izz="0.0004633"/>
+        <origin xyz="0.0 ${-reflect*0.0} -0.042127" rpy="0 0 0"/>
+        <!-- <origin xyz="-0.006788 ${-reflect*0.000020} -0.042127" rpy="0 0 0"/> -->
+        <mass value="1.0"/>
+        <!-- <mass value="1.015338978"/> -->
+        <inertia ixx="2.6324E-4" ixy="${-reflect*0.0}" ixz="7.4E-6" iyy="0.000571" iyz="${-reflect*0}" izz="4.633E-4"/>
+        <!-- REVISAR! -->
+        <!-- <inertia ixx="2.6324E-7" ixy="${-reflect*0.0}" ixz="7.4E-9" iyy="0.000000571" iyz="${-reflect*0}" izz="4.633E-7"/> -->
       </inertial>
       <xacro:insert_visualization_ankle_roll side="${side}" reflect="${reflect}"/>
@@ -127,6 +143,8 @@
       <inertial>
         <origin xyz="0.022629 ${-reflect*0.002448} 0.011325" rpy="0 0 0"/>
-        <mass value="2.884061022"/>
-        <inertia ixx="0.006699" ixy="${-reflect*-0.00009295}" ixz="0.00009066" iyy="0.00169929" iyz="${-reflect*0.00000708}" izz="0.00228359"/>
+        <!-- <origin xyz="0.022629 ${-reflect*0.002448} 0.011325" rpy="0 0 0"/> -->
+        <mass value="1.0"/>
+        <!-- <mass value="2.884061022"/> -->
+        <inertia ixx="6.699E-4" ixy="${-reflect*-0.000093}" ixz="9.066E-5" iyy="1.69929E-3" iyz="${-reflect*7.08E-6}" izz="2.28359E-3"/>
       </inertial>
       <xacro:insert_visualization_foot side="${side}" reflect="${reflect}"/>

File: teo_description/urdf/torso/torso.urdf.xacro (robot description, xacro)
@@ -9,4 +9,5 @@
 <robot name="teo" xmlns:xacro="http://ros.org/wiki/xacro">
 <!-- *** TEO TORSO PARAMETERS -->
+  <xacro:property name="prop_torso_kg_motor_vol_unit" value="6229.073482" /> <!-- Relation Kg - Volume Unit -->
 <!-- Link lengths -->
 	<xacro:property name="waist_link1" value="0.0" />
@@ -43,11 +44,20 @@
   <link name="waist" >
     <inertial>
-      <origin xyz="-0.011195 0.000002 0.030531" rpy="0 0 0"/>
+      <origin xyz="0.0 0.0 0.030531" rpy="0 0 0"/>
+      <!-- <origin xyz="-0.011195 0.000002 0.030531" rpy="0 0 0"/> -->
+      <mass value="1.0"/>
+      <inertia
+        ixx="1.672965e-2" ixy="-4.1e-7" ixz="-4.0359e-4"
+        iyy="8.75441e-3" iyz="8.0e-8"
+        izz="0.020584" />
+    </inertial>
+<!--     <inertial>
+      <origin xyz="0.0 0.0 0.57136" rpy="0 0 0"/>
       <mass value="5.7044"/>
       <inertia
-			  ixx="0.019" ixy="0.000" ixz="0.000"
-				iyy="0.018" iyz="0.000"
-				izz="0.008" />
-    </inertial>
+        ixx="0.019" ixy="0.000" ixz="0.000"
+        iyy="0.018" iyz="0.000"
+        izz="0.008" />
+    </inertial> -->
 <!--     <inertial>
       <origin xyz="-0.011195 0.000002 0.030531" rpy="0 0 0"/>
@@ -62,25 +72,32 @@
   <link name="waist_yaw_link" >
     <inertial>
-      <origin xyz="0 0 0" rpy="0 0 0"/>
-      <mass value="0.1"/>
+      <origin xyz="0.0 0.0 -0.024630" rpy="0 0 0"/>
+      <!-- <origin xyz="-0.004091 -0.001037 -0.024630" rpy="0 0 0"/> -->
+      <!-- <mass value="${prop_torso_kg_motor_vol_unit*0.000142}"/> -->
+      <mass value="1.0"/>
       <inertia
-			  ixx="0.1000" ixy="0.000" ixz="0.000"
-				iyy="0.1000" iyz="0.000"
-				izz="0.1000" />
+			  ixx="0.66667" ixy="-0.25" ixz="-0.25"
+				iyy="0.66667" iyz="-0.25"
+				izz="0.66667" />
+<!--       <inertia
+        ixx="2.8026e-4" ixy="-2.9e-7" ixz="-4.22e-6"
+        iyy="1.275e-4" iyz="4.4e-7"
+        izz="2.0857e-4" /> -->
     </inertial>
     <xacro:insert_visualization_waist_yaw/>
   </link>
-<!--   <link name="waist_pitch_link" >
+  <link name="waist_pitch_link" >
     <inertial>
-      <origin xyz="0 0 0" rpy="0 0 0"/>
-      <mass value="20.0"/>
+      <origin xyz="0.0 0.0 0.221233" rpy="0 0 0"/>
+      <!-- <origin xyz="0.038788 -0.000008 0.221233" rpy="0 0 0"/> -->
+      <mass value="1.0"/>
       <inertia
-        ixx="0.34286" ixy="0.000016480" ixz="-0.0012113"
-        iyy="0.12925" iyz="0.000093038"
-        izz="0.26900" />
+        ixx="0.3563817" ixy="-5.5E-6" ixz="-0.014295"
+        iyy="0.1422663" iyz="-2.205e-5"
+        izz="0.2704611" />
     </inertial>
     <xacro:insert_visualization_waist_pitch/>
     <xacro:insert_visualization_torso/>
-  </link> -->
+  </link>
   <!-- Joints -->
   <joint name="waist_yaw" type="revolute">
@@ -91,5 +108,5 @@
     <limit velocity="${waist_yaw_velocity}" effort="${waist_yaw_effort}" lower="${waist_yaw_lower}" upper="${waist_yaw_upper}"/>
   </joint>
-<!--   <joint name="waist_pitch" type="revolute">
+  <joint name="waist_pitch" type="revolute">
     <parent link="waist_yaw_link"/>
     <child link="waist_pitch_link"/>
@@ -97,6 +114,6 @@
     <axis xyz="0 1 0"/>
     <limit velocity="${waist_pitch_velocity}" effort="${waist_pitch_effort}" lower="${waist_pitch_lower}" upper="${waist_pitch_upper}"/>
-  </joint> -->
+  </joint>
   <xacro:waist_joint_simple_transmission axis="yaw" reduction="${waist_yaw_reduction}"/>
-  <!-- <xacro:waist_joint_simple_transmission axis="pitch" reduction="${waist_pitch_reduction}"/> -->
+  <xacro:waist_joint_simple_transmission axis="pitch" reduction="${waist_pitch_reduction}"/>
 </robot>
