Commit message: xacro now considers teo's platform

File: teo_description/robots/teo_humanoid.urdf.xacro (robot description, xacro)
@@ -11,16 +11,19 @@
 -->
 <robot name="teo" xmlns:xacro="http://ros.org/wiki/xacro">
+  <!-- TEO parameters -->
+  <xacro:property name="use_static_platform" value="false" />
   <!-- TEO structure -->
   <xacro:include filename="$(find teo_description)/urdf/teo_structure.urdf.xacro" />
   <!-- TEO visualization -->
   <!--xacro:if value="$(arg simple_vis)">
-    <xacro:include filename="$(find teo_description)/urdf/simple_visual.xacro" />
+    <xacro:include filename="$(find teo_description)/urdf/others/simple_visual.xacro" />
   </xacro:if-->
   <!--xacro:unless complete_vis="$(arg complete_vis)">
-    <xacro:include filename="$(find teo_description)/urdf/visualization.xacro" />
+    <xacro:include filename="$(find teo_description)/urdf/others/visualization.xacro" />
   </xacro:unless-->
-  <!--xacro:include filename="$(find teo_description)/urdf/simple_visual.xacro" /-->
-  <xacro:include filename="$(find teo_description)/urdf/torso/torso_simple_vis.urdf.xacro" />
-  <xacro:include filename="$(find teo_description)/urdf/legs/legs_simple_vis.urdf.xacro" />
-  <xacro:include filename="$(find teo_description)/urdf/arms/arms_simple_vis.urdf.xacro" />
+  <!--xacro:include filename="$(find teo_description)/urdf/visual.xacro" /-->
+  <xacro:include filename="$(find teo_description)/urdf/others/teo_colors.xacro" />
+  <xacro:include filename="$(find teo_description)/urdf/torso/torso_vis.urdf.xacro" />
+  <xacro:include filename="$(find teo_description)/urdf/legs/legs_vis.urdf.xacro" />
+  <xacro:include filename="$(find teo_description)/urdf/arms/arms_vis.urdf.xacro" />
 </robot>

File: teo_description/robots/teo_humanoid_simple_vis.urdf.xacro (robot description, xacro)
@@ -15,13 +15,12 @@
   <!-- TEO visualization -->
   <!--xacro:if value="$(arg simple_vis)">
-    <xacro:include filename="$(find teo_description)/urdf/simple_visual.xacro" />
+    <xacro:include filename="$(find teo_description)/urdf/others/simple_visual.xacro" />
   </xacro:if-->
   <!--xacro:unless complete_vis="$(arg complete_vis)">
-    <xacro:include filename="$(find teo_description)/urdf/visualization.xacro" />
+    <xacro:include filename="$(find teo_description)/urdf/others/visualization.xacro" />
   </xacro:unless-->
-  <!--xacro:include filename="$(find teo_description)/urdf/visual.xacro" /-->
-  <xacro:include filename="$(find teo_description)/urdf/others/teo_colors.xacro" />
-  <xacro:include filename="$(find teo_description)/urdf/torso/torso_vis.urdf.xacro" />
-  <xacro:include filename="$(find teo_description)/urdf/legs/legs_vis.urdf.xacro" />
-  <xacro:include filename="$(find teo_description)/urdf/arms/arms_vis.urdf.xacro" />
+  <!--xacro:include filename="$(find teo_description)/urdf/simple_visual.xacro" /-->
+  <xacro:include filename="$(find teo_description)/urdf/torso/torso_simple_vis.urdf.xacro" />
+  <xacro:include filename="$(find teo_description)/urdf/legs/legs_simple_vis.urdf.xacro" />
+  <xacro:include filename="$(find teo_description)/urdf/arms/arms_simple_vis.urdf.xacro" />
 </robot>

File: teo_description/urdf/arms/arms_vis.urdf.xacro (robot description, xacro)
@@ -15,8 +15,8 @@
     </visual>
     <collision>
+      <origin rpy="0 0 0" xyz="0 0 0"/>
       <geometry>
-        <box size="0.1 ${arm_link1} 0.1"/>
+        <mesh filename="package://teo_description/meshes/arms/${side}_shoulder_pitch.stl"/>
       </geometry>
-      <origin rpy="0 0 0" xyz="0 0 0"/>
     </collision>
   </xacro:macro>
@@ -30,8 +30,8 @@
     </visual>
     <collision>
+      <origin rpy="0 0 0" xyz="0 0 0"/>
       <geometry>
-        <box size="0.1 ${arm_link1} 0.1"/>
+        <mesh filename="package://teo_description/meshes/arms/${side}_shoulder_roll.stl"/>
       </geometry>
-      <origin rpy="0 0 0" xyz="0 0 0"/>
     </collision>
   </xacro:macro>
@@ -44,4 +44,10 @@
       <material name="teoGray"/>
     </visual>
+    <collision>
+      <origin rpy="0 0 0" xyz="0 0 -0.12126"/>
+      <geometry>
+        <mesh filename="package://teo_description/meshes/arms/${side}_shoulder_yaw.stl"/>
+      </geometry>
+    </collision>
     <visual>
       <origin rpy="0 0 0" xyz="0 0 -0.27651"/>
@@ -51,4 +57,10 @@
       <material name="teoGray"/>
     </visual>
+    <collision>
+      <origin rpy="0 0 0" xyz="0 0 -0.27651"/>
+      <geometry>
+        <mesh filename="package://teo_description/meshes/arms/${side}_humerus.stl"/>
+      </geometry>
+    </collision>
     <visual>
       <origin rpy="0 0 0" xyz="0 0 -0.28351"/>
@@ -59,8 +71,8 @@
     </visual>
     <collision>
+      <origin rpy="0 0 0" xyz="0 0 -0.28351"/>
       <geometry>
-        <box size="0.08 0.08 ${arm_link2}"/>
+        <mesh filename="package://teo_description/meshes/arms/${side}_union_humerus_elbow.stl"/>
       </geometry>
-      <origin rpy="0 0 0" xyz="0 0 -${arm_link2/2}"/>
     </collision>
   </xacro:macro>
@@ -73,4 +85,10 @@
       <material name="teoGray"/>
     </visual>
+    <collision>
+      <origin rpy="0 0 0" xyz="0 0 0"/>
+      <geometry>
+        <mesh filename="package://teo_description/meshes/arms/${side}_elbow_pitch.stl"/>
+      </geometry>
+    </collision>
     <visual>
       <origin rpy="0 0 0" xyz="0 0 -0.11324"/>
@@ -78,5 +96,12 @@
         <mesh filename="package://teo_description/meshes/arms/${side}_elbow_link.stl"/>
       </geometry>
+      <material name="teoGray"/>
     </visual>
+    <collision>
+      <origin rpy="0 0 0" xyz="0 0 -0.11324"/>
+      <geometry>
+        <mesh filename="package://teo_description/meshes/arms/${side}_elbow_link.stl"/>
+      </geometry>
+    </collision>
     <visual>
       <origin rpy="0 0 0" xyz="0 0 -0.11324"/>
@@ -87,8 +112,8 @@
     </visual>
     <collision>
+      <origin rpy="0 0 0" xyz="0 0 -0.11324"/>
       <geometry>
-        <box size="0.06 0.06 ${arm_link3}"/>
+        <mesh filename="package://teo_description/meshes/arms/${side}_union_elbow_wrist.stl"/>
       </geometry>
-      <origin rpy="0 0 0" xyz="0 0 -${arm_link3/2}"/>
     </collision>
   </xacro:macro>
@@ -102,8 +127,8 @@
     </visual>
     <collision>
+      <origin rpy="0 0 0" xyz="0 0 0"/>
       <geometry>
-        <box size="0.03 0.03 0.03"/>
+        <mesh filename="package://teo_description/meshes/arms/${side}_wrist_yaw.stl"/>
       </geometry>
-      <origin rpy="0 0 0" xyz="0 0 -0.015"/>
     </collision>
   </xacro:macro>
@@ -116,4 +141,10 @@
       <material name="teoGray"/>
     </visual>
+    <collision>
+      <origin rpy="0 0 0" xyz="0 0 0"/>
+      <geometry>
+        <mesh filename="package://teo_description/meshes/arms/${side}_wrist_pitch.stl"/>
+      </geometry>
+    </collision>
     <visual>
       <origin rpy="0 0 0" xyz="0 0 -0.056"/>
@@ -123,4 +154,10 @@
       <material name="teoGray"/>
     </visual>
+    <collision>
+      <origin rpy="0 0 0" xyz="0 0 -0.056"/>
+      <geometry>
+        <mesh filename="package://teo_description/meshes/arms/${side}_wrist_sensorFT.stl"/>
+      </geometry>
+    </collision>
     <visual>
       <origin rpy="0 0 0" xyz="0 0 -0.056"/>
@@ -131,8 +168,8 @@
     </visual>
     <collision>
+      <origin rpy="0 0 0" xyz="0 0 -0.056"/>
       <geometry>
-        <box size="0.03 0.03 0.03"/>
+        <mesh filename="package://teo_description/meshes/arms/${side}_hand.stl"/>
       </geometry>
-      <origin rpy="0 0 0" xyz="0 0 -0.015"/>
     </collision>
   </xacro:macro>

File: teo_description/urdf/legs/legs_vis.urdf.xacro (robot description, xacro)
@@ -15,7 +15,7 @@
     </visual>
     <collision>
-      <origin xyz="0 0 0.045" rpy="0 1.571 0"/>
+      <origin rpy="0 0 0" xyz="0 0 0"/>
       <geometry>
-        <cylinder radius="0.045" length="0.13"/>
+        <mesh filename="package://teo_description/meshes/legs/${side}_hip_yaw.stl"/>
       </geometry>
     </collision>
@@ -29,4 +29,10 @@
       <material name="teoGray"/>
     </visual>
+    <collision>
+      <origin rpy="0 0 0" xyz="0 0 0"/>
+      <geometry>
+        <mesh filename="package://teo_description/meshes/legs/${side}_hip_pitch.stl"/>
+      </geometry>
+    </collision>
   </xacro:macro>
   <xacro:macro name="insert_visualization_femur_link" params="side reflect">
@@ -39,8 +45,8 @@
     </visual>
     <collision>
+      <origin rpy="0 0 0" xyz="0 0 0"/>
       <geometry>
-        <box size="0.1 0.1 ${leg_link2}"/>
+        <mesh filename="package://teo_description/meshes/legs/${side}_femur.stl"/>
       </geometry>
-      <origin rpy="0 0 0" xyz="0 0 -${leg_link2/2}"/>
     </collision>
   </xacro:macro>
@@ -54,8 +60,8 @@
     </visual>
     <collision>
+      <origin rpy="0 0 0" xyz="0.0 0.0 0.0"/>
       <geometry>
-        <box size="0.05 ${leg_link4} 0.05"/>
+        <mesh filename="package://teo_description/meshes/legs/${side}_tibia.stl"/>
       </geometry>
-      <origin rpy="0 0 0" xyz="0 ${reflect*-leg_link4} -${leg_link3-0.05/2}"/>
     </collision>
   </xacro:macro>
@@ -68,4 +74,10 @@
       <material name="teoGray"/>
     </visual>
+    <collision>
+      <origin rpy="0 0 0" xyz="0 0 0"/>
+      <geometry>
+        <mesh filename="package://teo_description/meshes/legs/${side}_ankle_pitch.stl"/>
+      </geometry>
+    </collision>
   </xacro:macro>
   <xacro:macro name="insert_visualization_ankle_roll" params="side reflect">
@@ -77,4 +89,10 @@
       <material name="teoGray"/>
     </visual>
+    <collision>
+      <origin rpy="0 0 0" xyz="0 0 0"/>
+      <geometry>
+        <mesh filename="package://teo_description/meshes/legs/${side}_ankle_roll.stl"/>
+      </geometry>
+    </collision>
     <visual>
       <origin rpy="0 0 0" xyz="0 0 -0.073"/>
@@ -83,4 +101,10 @@
       </geometry>
     </visual>
+    <collision>
+      <origin rpy="0 0 0" xyz="0 0 -0.073"/>
+      <geometry>
+        <mesh filename="package://teo_description/meshes/legs/${side}_ankle_sensorFT.stl"/>
+      </geometry>
+    </collision>
   </xacro:macro>
   <xacro:macro name="insert_visualization_foot" params="side reflect">
@@ -93,9 +117,8 @@
     </visual>
     <collision>
+      <origin rpy="0 0 0" xyz="0 0 0"/>
       <geometry>
-        <!-- <box size="0.08 0.08 ${leg_link5}"/> -->
-        <box size="0.245438 0.139979 0.019500"/>
+        <mesh filename="package://teo_description/meshes/legs/${side}_foot.stl"/>
       </geometry>
-      <origin rpy="0 0 0" xyz="0.05 0 0.00975"/>
     </collision>
   </xacro:macro>
@@ -108,4 +131,10 @@
       <material name="teoBlue"/>
     </visual>
+    <collision>
+      <origin rpy="0 0 0" xyz="0 0 0"/>
+      <geometry>
+        <mesh filename="package://teo_description/meshes/legs/${side}_union_sensorFT_foot.stl"/>
+      </geometry>
+    </collision>
   </xacro:macro>
   <xacro:macro name="insert_visualization_sole" params="side reflect">

File: teo_description/urdf/teo_structure.urdf.xacro (robot description, xacro)
@@ -13,31 +13,33 @@
 <!-- Include useful constants -->
 <xacro:include filename="$(find teo_description)/urdf/others/teo_constants.xacro" />
+<!-- Include joint transmissions -->
 <xacro:include filename="$(find teo_description)/urdf/others/teo_transmission.xacro" />
-<!-- **** Torso **** -->
-  <!-- base_link is rigidly attached to the robot root body.
-  It is recommended to choose the robot waist as its root body -->
-  <link name="base_link" />
-<!--***************
-    **** JOINTS ****
-    ***************-->
+<!-- Use TEO platform -->
+<xacro:if value="${use_static_platform}">
+  <xacro:include filename="$(find teo_description)/urdf/others/teo_platform.xacro" />
+</xacro:if>
+<!-- **** Torso - base_link **** -->
+<!-- base_link is rigidly attached to the robot root body.
+It is recommended to choose the robot waist as its root body -->
+<link name="base_link" />
 <!-- **** Fictitious joints **** -->
-  <joint name="base_joint" type="fixed">
-    <child link="waist"/>
-    <parent link="base_link"/>
-    <origin xyz="0 0 0" rpy="0 0 0" />
-  </joint>
+<joint name="base_joint" type="fixed">
+  <parent link="base_link"/>
+  <child link="waist"/>
+  <origin xyz="0 0 0" rpy="0 0 0" />
+</joint>
  <!-- Definitions of parts of the robot body -->
  <xacro:include filename="$(find teo_description)/urdf/torso/torso.urdf.xacro" />
  <xacro:include filename="$(find teo_description)/urdf/legs/leg.urdf.xacro" />
- <xacro:include filename="$(find teo_description)/urdf/arms/arm.urdf.xacro" />
+ <!-- <xacro:include filename="$(find teo_description)/urdf/arms/arm.urdf.xacro" /> -->
 <!--****************
     **** GAZEBO ****
     ****************-->
   <!-- Import all Gazebo-customization elements, including Gazebo colors -->
-  <xacro:include filename="$(find teo_description)/urdf/teo_humanoid.gazebo.xacro" />
+  <xacro:include filename="$(find teo_description)/urdf/teo_structure.gazebo.xacro" />
   <xacro:gazebo_torso/>
   <xacro:gazebo_legs_links side="l" reflect="1"/>
   <xacro:gazebo_legs_links side="r" reflect="-1"/>
-  <xacro:gazebo_arms_links side="l" reflect="1"/>
-  <xacro:gazebo_arms_links side="r" reflect="-1"/>
+<!--   <xacro:gazebo_arms_links side="l" reflect="1"/>
+  <xacro:gazebo_arms_links side="r" reflect="-1"/> -->
 </robot>

File: teo_description/urdf/torso/torso.urdf.xacro (robot description, xacro)
@@ -63,5 +63,5 @@
     <xacro:insert_visualization_waist_yaw/>
   </link>
-  <link name="waist_pitch_link" >
+<!--   <link name="waist_pitch_link" >
     <inertial>
       <origin xyz="0 0 0" rpy="0 0 0"/>
@@ -74,5 +74,5 @@
     <xacro:insert_visualization_waist_pitch/>
     <xacro:insert_visualization_torso/>
-  </link>
+  </link> -->
   <!-- Joints -->
   <joint name="waist_yaw" type="revolute">
@@ -83,5 +83,5 @@
     <limit velocity="${waist_yaw_velocity}" effort="${waist_yaw_effort}" lower="${waist_yaw_lower}" upper="${waist_yaw_upper}"/>
   </joint>
-  <joint name="waist_pitch" type="revolute">
+<!--   <joint name="waist_pitch" type="revolute">
     <parent link="waist_yaw_link"/>
     <child link="waist_pitch_link"/>
@@ -89,6 +89,6 @@
     <axis xyz="0 1 0"/>
     <limit velocity="${waist_pitch_velocity}" effort="${waist_pitch_effort}" lower="${waist_pitch_lower}" upper="${waist_pitch_upper}"/>
-  </joint>
-    <xacro:waist_joint_simple_transmission axis="yaw" reduction="${waist_yaw_reduction}"/>
-    <xacro:waist_joint_simple_transmission axis="pitch" reduction="${waist_pitch_reduction}"/>
+  </joint> -->
+  <xacro:waist_joint_simple_transmission axis="yaw" reduction="${waist_yaw_reduction}"/>
+  <!-- <xacro:waist_joint_simple_transmission axis="pitch" reduction="${waist_pitch_reduction}"/> -->
 </robot>

File: teo_description/urdf/torso/torso_vis.urdf.xacro (robot description, xacro)
@@ -15,8 +15,7 @@
     </visual>
     <collision>
-      <origin xyz="0 0 0.025" rpy="0 0 0"/>
+      <origin xyz="0 0 -0.001" rpy="0 0 0"/>
       <geometry>
-         <!--sphere radius="1.0"/-->
-         <cylinder radius="0.02" length="0.06"/>
+        <mesh filename="package://teo_description/meshes/torso/waist-yaw.stl"/>
       </geometry>
     </collision>
@@ -31,9 +30,9 @@
     </visual>
     <collision>
-      <origin xyz="0 0 0" rpy="${pi_2} 0 0"/>
+      <origin xyz="0 0 0" rpy="0 0 0"/>
       <geometry>
-        <!--sphere radius="1.0"/-->
-        <cylinder radius="0.02" length="0.06"/>
+        <mesh filename="package://teo_description/meshes/torso/waist-pitch.stl"/>
       </geometry>
+      <material name="teoGray"/>
     </collision>
   </xacro:macro>
@@ -46,4 +45,10 @@
       <material name="teoGray"/>
     </visual>
+    <collision>
+      <origin xyz="0 0 ${torso_link2}" rpy="0 0 0"/>
+      <geometry>
+        <mesh filename="package://teo_description/meshes/torso/torso.stl"/>
+      </geometry>
+    </collision>
     <visual>
       <origin xyz="0 0.25486 ${torso_link2+chest_link2}" rpy="0 0 0"/>
@@ -53,4 +58,10 @@
       <material name="teoGray"/>
     </visual>
+    <collision>
+      <origin xyz="0 0.25486 ${torso_link2+chest_link2}" rpy="0 0 0"/>
+      <geometry>
+        <mesh filename="package://teo_description/meshes/torso/L-torso-shoulder.stl"/>
+      </geometry>
+    </collision>
     <visual>
       <origin xyz="0 -0.25486 ${torso_link2+chest_link2}" rpy="0 0 0"/>
@@ -60,4 +71,10 @@
       <material name="LightGrey"/>
     </visual>
+    <collision>
+      <origin xyz="0 -0.25486 ${torso_link2+chest_link2}" rpy="0 0 0"/>
+      <geometry>
+        <mesh filename="package://teo_description/meshes/torso/R-torso-shoulder.stl"/>
+      </geometry>
+    </collision>
     <visual>
       <origin xyz="0 0 0.346" rpy="0 0 0"/>
@@ -67,4 +84,10 @@
       <material name="LightGrey"/>
     </visual>
+    <collision>
+      <origin xyz="0 0 0.346" rpy="0 0 0"/>
+      <geometry>
+        <mesh filename="package://teo_description/meshes/torso/neck.stl"/>
+      </geometry>
+    </collision>
     <visual>
       <origin xyz="0 0 0.434" rpy="0 0 0"/>
@@ -75,7 +98,7 @@
     </visual>
     <collision>
-      <origin xyz="0 0 0.1" rpy="0 0 0"/>
+      <origin xyz="0 0 0.434" rpy="0 0 0"/>
       <geometry>
-        <box size="0.18 0.42 0.292"/>
+        <mesh filename="package://teo_description/meshes/torso/head.stl"/>
       </geometry>
     </collision>
@@ -89,4 +112,10 @@
       <material name="teoBlack"/>
     </visual>
+    <collision>
+      <origin xyz="0 0 0" rpy="0 0 0"/>
+      <geometry>
+        <mesh filename="package://teo_description/meshes/torso/waist-base.stl"/>
+      </geometry>
+    </collision>
     <visual>
       <origin xyz="0 0 0.07336" rpy="0 0 0"/>
@@ -96,4 +125,10 @@
       <material name="teoGray"/>
     </visual>
+    <collision>
+      <origin xyz="0 0 0.07336" rpy="0 0 0"/>
+      <geometry>
+        <mesh filename="package://teo_description/meshes/torso/waist-link.stl"/>
+      </geometry>
+    </collision>
   </xacro:macro>
 </robot>
